Commit message: Fixed bug in importing limits

File: generated/gazebo_models/iCubGenova01/icub_simulation.urdf (robot description, URDF)
Before this commit: robot test_icub, 46 links, 45 joints
Joints:
- joint l_ankle_pitch: limit (none) -> lower=-0.733038 upper=0.366519 effort=24 velocity=100; type continuous -> revolute
- joint l_ankle_roll: limit (none) -> lower=-0.418879 upper=0.418879 effort=11 velocity=100; type continuous -> revolute
- joint l_hip_pitch: limit (none) -> lower=-0.767945 upper=2.30383 effort=84 velocity=100; type continuous -> revolute
- joint l_hip_roll: limit (none) -> lower=-2.07694 upper=0.296706 effort=84 velocity=100; type continuous -> revolute
- joint l_hip_yaw: limit (none) -> lower=-1.37881 upper=1.37881 effort=40 velocity=100; type continuous -> revolute
- joint l_knee: limit (none) -> lower=-2.18166 upper=0.401426 effort=30 velocity=100; type continuous -> revolute
- joint l_shoulder_pitch: limit (none) -> lower=-1.65806 upper=0.0872665 effort=84 velocity=100; type continuous -> revolute
- joint l_shoulder_roll: limit (none) -> lower=0 upper=2.80649 effort=84 velocity=100; type continuous -> revolute
- joint l_shoulder_yaw: limit (none) -> lower=-0.645772 upper=1.74533 effort=34 velocity=100; type continuous -> revolute
- joint l_wrist_pitch: limit (none) -> lower=-0.436332 upper=0.436332 effort=0.65 velocity=100; type continuous -> revolute
- joint neck_pitch: limit (none) -> lower=-0.698132 upper=0.523599 effort=20 velocity=100; type continuous -> revolute
- joint neck_roll: limit (none) -> lower=-1.22173 upper=1.0472 effort=20 velocity=100; type continuous -> revolute
- joint neck_yaw: limit (none) -> lower=-0.959931 upper=0.959931 effort=20 velocity=100; type continuous -> revolute
- joint r_ankle_pitch: limit (none) -> lower=-0.733038 upper=0.366519 effort=24 velocity=100; type continuous -> revolute
- joint r_ankle_roll: limit (none) -> lower=-0.418879 upper=0.418879 effort=11 velocity=100; type continuous -> revolute
- joint r_hip_pitch: limit (none) -> lower=-0.767945 upper=2.30383 effort=84 velocity=100; type continuous -> revolute
- joint r_hip_roll: limit (none) -> lower=-2.07694 upper=0.296706 effort=84 velocity=100; type continuous -> revolute
- joint r_hip_yaw: limit (none) -> lower=-1.37881 upper=1.37881 effort=40 velocity=100; type continuous -> revolute
- joint r_knee: limit (none) -> lower=-2.18166 upper=0.401426 effort=30 velocity=100; type continuous -> revolute
- joint r_shoulder_pitch: limit (none) -> lower=-1.65806 upper=0.0872665 effort=84 velocity=100; type continuous -> revolute
- joint r_shoulder_roll: limit (none) -> lower=0 upper=2.80649 effort=84 velocity=100; type continuous -> revolute
- joint r_shoulder_yaw: limit (none) -> lower=-0.645772 upper=1.74533 effort=34 velocity=100; type continuous -> revolute
- joint r_wrist_pitch: limit (none) -> lower=-0.436332 upper=0.436332 effort=0.65 velocity=100; type continuous -> revolute
- joint torso_pitch: limit (none) -> lower=-0.383972 upper=1.46608 effort=36 velocity=100; type continuous -> revolute
- joint torso_roll: limit (none) -> lower=-0.680678 upper=0.680678 effort=80 velocity=100; type continuous -> revolute
- joint torso_yaw: limit (none) -> lower=-1.02974 upper=1.02974 effort=80 velocity=100; type continuous -> revolute

File: generated/gazebo_models/iCubGenova03/icub_simulation.urdf (robot description, URDF)
Before this commit: robot test_icub, 46 links, 45 joints
Joints:
- joint l_ankle_pitch: limit (none) -> lower=-0.733038 upper=0.366519 effort=24 velocity=100; type continuous -> revolute
- joint l_ankle_roll: limit (none) -> lower=-0.418879 upper=0.418879 effort=11 velocity=100; type continuous -> revolute
- joint l_hip_pitch: limit (none) -> lower=-0.767945 upper=2.30383 effort=84 velocity=100; type continuous -> revolute
- joint l_hip_roll: limit (none) -> lower=-2.07694 upper=0.296706 effort=84 velocity=100; type continuous -> revolute
- joint l_hip_yaw: limit (none) -> lower=-1.37881 upper=1.37881 effort=40 velocity=100; type continuous -> revolute
- joint l_knee: limit (none) -> lower=-2.18166 upper=0.401426 effort=30 velocity=100; type continuous -> revolute
- joint l_shoulder_pitch: limit (none) -> lower=-1.65806 upper=0.0872665 effort=84 velocity=100; type continuous -> revolute
- joint l_shoulder_roll: limit (none) -> lower=0 upper=2.80649 effort=84 velocity=100; type continuous -> revolute
- joint l_shoulder_yaw: limit (none) -> lower=-0.645772 upper=1.74533 effort=34 velocity=100; type continuous -> revolute
- joint l_wrist_pitch: limit (none) -> lower=-0.436332 upper=0.436332 effort=0.65 velocity=100; type continuous -> revolute
- joint neck_pitch: limit (none) -> lower=-0.698132 upper=0.523599 effort=20 velocity=100; type continuous -> revolute
- joint neck_roll: limit (none) -> lower=-1.22173 upper=1.0472 effort=20 velocity=100; type continuous -> revolute
- joint neck_yaw: limit (none) -> lower=-0.959931 upper=0.959931 effort=20 velocity=100; type continuous -> revolute
- joint r_ankle_pitch: limit (none) -> lower=-0.733038 upper=0.366519 effort=24 velocity=100; type continuous -> revolute
- joint r_ankle_roll: limit (none) -> lower=-0.418879 upper=0.418879 effort=11 velocity=100; type continuous -> revolute
- joint r_hip_pitch: limit (none) -> lower=-0.767945 upper=2.30383 effort=84 velocity=100; type continuous -> revolute
- joint r_hip_roll: limit (none) -> lower=-2.07694 upper=0.296706 effort=84 velocity=100; type continuous -> revolute
- joint r_hip_yaw: limit (none) -> lower=-1.37881 upper=1.37881 effort=40 velocity=100; type continuous -> revolute
- joint r_knee: limit (none) -> lower=-2.18166 upper=0.401426 effort=30 velocity=100; type continuous -> revolute
- joint r_shoulder_pitch: limit (none) -> lower=-1.65806 upper=0.0872665 effort=84 velocity=100; type continuous -> revolute
- joint r_shoulder_roll: limit (none) -> lower=0 upper=2.80649 effort=84 velocity=100; type continuous -> revolute
- joint r_shoulder_yaw: limit (none) -> lower=-0.645772 upper=1.74533 effort=34 velocity=100; type continuous -> revolute
- joint r_wrist_pitch: limit (none) -> lower=-0.436332 upper=0.436332 effort=0.65 velocity=100; type continuous -> revolute
- joint torso_pitch: limit (none) -> lower=-0.383972 upper=1.46608 effort=36 velocity=100; type continuous -> revolute
- joint torso_roll: limit (none) -> lower=-0.680678 upper=0.680678 effort=80 velocity=100; type continuous -> revolute
- joint torso_yaw: limit (none) -> lower=-1.02974 upper=1.02974 effort=80 velocity=100; type continuous -> revolute

File: generated/urdf/iCubGenova01/icub.urdf (robot description, URDF)
Before this commit: robot test_icub, 46 links, 45 joints
Joints:
- joint l_ankle_pitch: limit (none) -> lower=-0.733038 upper=0.366519 effort=24 velocity=100; type continuous -> revolute
- joint l_ankle_roll: limit (none) -> lower=-0.418879 upper=0.418879 effort=11 velocity=100; type continuous -> revolute
- joint l_hip_pitch: limit (none) -> lower=-0.767945 upper=2.30383 effort=84 velocity=100; type continuous -> revolute
- joint l_hip_roll: limit (none) -> lower=-2.07694 upper=0.296706 effort=84 velocity=100; type continuous -> revolute
- joint l_hip_yaw: limit (none) -> lower=-1.37881 upper=1.37881 effort=40 velocity=100; type continuous -> revolute
- joint l_knee: limit (none) -> lower=-2.18166 upper=0.401426 effort=30 velocity=100; type continuous -> revolute
- joint l_shoulder_pitch: limit (none) -> lower=-1.65806 upper=0.0872665 effort=84 velocity=100; type continuous -> revolute
- joint l_shoulder_roll: limit (none) -> lower=0 upper=2.80649 effort=84 velocity=100; type continuous -> revolute
- joint l_shoulder_yaw: limit (none) -> lower=-0.645772 upper=1.74533 effort=34 velocity=100; type continuous -> revolute
- joint l_wrist_pitch: limit (none) -> lower=-0.436332 upper=0.436332 effort=0.65 velocity=100; type continuous -> revolute
- joint neck_pitch: limit (none) -> lower=-0.698132 upper=0.523599 effort=20 velocity=100; type continuous -> revolute
- joint neck_roll: limit (none) -> lower=-1.22173 upper=1.0472 effort=20 velocity=100; type continuous -> revolute
- joint neck_yaw: limit (none) -> lower=-0.959931 upper=0.959931 effort=20 velocity=100; type continuous -> revolute
- joint r_ankle_pitch: limit (none) -> lower=-0.733038 upper=0.366519 effort=24 velocity=100; type continuous -> revolute
- joint r_ankle_roll: limit (none) -> lower=-0.418879 upper=0.418879 effort=11 velocity=100; type continuous -> revolute
- joint r_hip_pitch: limit (none) -> lower=-0.767945 upper=2.30383 effort=84 velocity=100; type continuous -> revolute
- joint r_hip_roll: limit (none) -> lower=-2.07694 upper=0.296706 effort=84 velocity=100; type continuous -> revolute
- joint r_hip_yaw: limit (none) -> lower=-1.37881 upper=1.37881 effort=40 velocity=100; type continuous -> revolute
- joint r_knee: limit (none) -> lower=-2.18166 upper=0.401426 effort=30 velocity=100; type continuous -> revolute
- joint r_shoulder_pitch: limit (none) -> lower=-1.65806 upper=0.0872665 effort=84 velocity=100; type continuous -> revolute
- joint r_shoulder_roll: limit (none) -> lower=0 upper=2.80649 effort=84 velocity=100; type continuous -> revolute
- joint r_shoulder_yaw: limit (none) -> lower=-0.645772 upper=1.74533 effort=34 velocity=100; type continuous -> revolute
- joint r_wrist_pitch: limit (none) -> lower=-0.436332 upper=0.436332 effort=0.65 velocity=100; type continuous -> revolute
- joint torso_pitch: limit (none) -> lower=-0.383972 upper=1.46608 effort=36 velocity=100; type continuous -> revolute
- joint torso_roll: limit (none) -> lower=-0.680678 upper=0.680678 effort=80 velocity=100; type continuous -> revolute
- joint torso_yaw: limit (none) -> lower=-1.02974 upper=1.02974 effort=80 velocity=100; type continuous -> revolute

File: generated/urdf/iCubGenova03/icub.urdf (robot description, URDF)
Before this commit: robot test_icub, 46 links, 45 joints
Joints:
- joint l_ankle_pitch: limit (none) -> lower=-0.733038 upper=0.366519 effort=24 velocity=100; type continuous -> revolute
- joint l_ankle_roll: limit (none) -> lower=-0.418879 upper=0.418879 effort=11 velocity=100; type continuous -> revolute
- joint l_hip_pitch: limit (none) -> lower=-0.767945 upper=2.30383 effort=84 velocity=100; type continuous -> revolute
- joint l_hip_roll: limit (none) -> lower=-2.07694 upper=0.296706 effort=84 velocity=100; type continuous -> revolute
- joint l_hip_yaw: limit (none) -> lower=-1.37881 upper=1.37881 effort=40 velocity=100; type continuous -> revolute
- joint l_knee: limit (none) -> lower=-2.18166 upper=0.401426 effort=30 velocity=100; type continuous -> revolute
- joint l_shoulder_pitch: limit (none) -> lower=-1.65806 upper=0.0872665 effort=84 velocity=100; type continuous -> revolute
- joint l_shoulder_roll: limit (none) -> lower=0 upper=2.80649 effort=84 velocity=100; type continuous -> revolute
- joint l_shoulder_yaw: limit (none) -> lower=-0.645772 upper=1.74533 effort=34 velocity=100; type continuous -> revolute
- joint l_wrist_pitch: limit (none) -> lower=-0.436332 upper=0.436332 effort=0.65 velocity=100; type continuous -> revolute
- joint neck_pitch: limit (none) -> lower=-0.698132 upper=0.523599 effort=20 velocity=100; type continuous -> revolute
- joint neck_roll: limit (none) -> lower=-1.22173 upper=1.0472 effort=20 velocity=100; type continuous -> revolute
- joint neck_yaw: limit (none) -> lower=-0.959931 upper=0.959931 effort=20 velocity=100; type continuous -> revolute
- joint r_ankle_pitch: limit (none) -> lower=-0.733038 upper=0.366519 effort=24 velocity=100; type continuous -> revolute
- joint r_ankle_roll: limit (none) -> lower=-0.418879 upper=0.418879 effort=11 velocity=100; type continuous -> revolute
- joint r_hip_pitch: limit (none) -> lower=-0.767945 upper=2.30383 effort=84 velocity=100; type continuous -> revolute
- joint r_hip_roll: limit (none) -> lower=-2.07694 upper=0.296706 effort=84 velocity=100; type continuous -> revolute
- joint r_hip_yaw: limit (none) -> lower=-1.37881 upper=1.37881 effort=40 velocity=100; type continuous -> revolute
- joint r_knee: limit (none) -> lower=-2.18166 upper=0.401426 effort=30 velocity=100; type continuous -> revolute
- joint r_shoulder_pitch: limit (none) -> lower=-1.65806 upper=0.0872665 effort=84 velocity=100; type continuous -> revolute
- joint r_shoulder_roll: limit (none) -> lower=0 upper=2.80649 effort=84 velocity=100; type continuous -> revolute
- joint r_shoulder_yaw: limit (none) -> lower=-0.645772 upper=1.74533 effort=34 velocity=100; type continuous -> revolute
- joint r_wrist_pitch: limit (none) -> lower=-0.436332 upper=0.436332 effort=0.65 velocity=100; type continuous -> revolute
- joint torso_pitch: limit (none) -> lower=-0.383972 upper=1.46608 effort=36 velocity=100; type continuous -> revolute
- joint torso_roll: limit (none) -> lower=-0.680678 upper=0.680678 effort=80 velocity=100; type continuous -> revolute
- joint torso_yaw: limit (none) -> lower=-1.02974 upper=1.02974 effort=80 velocity=100; type continuous -> revolute

Commit message: Fixed difference in joint naming between genoa urdf models and paris

File: generated/gazebo_models/iCubGenova01/icub_simulation.urdf (robot description, URDF)
Before this commit: robot test_icub, 46 links, 45 joints
Joints:
- joint l_elbow: limit (none) -> lower=0.0959931 upper=1.85005 effort=20 velocity=100; type continuous -> revolute
- joint l_wrist_pitch: limit lower=-0.436332 upper=0.436332 effort=0.65 velocity=100 -> lower=-1.13446 upper=0.174533 effort=0.65 velocity=100
- joint l_wrist_prosup: limit (none) -> lower=-0.872665 upper=0.872665 effort=0.45 velocity=100; type continuous -> revolute
- joint l_wrist_yaw: limit (none) -> lower=-0.436332 upper=0.436332 effort=0.65 velocity=100; type continuous -> revolute
- joint r_elbow: limit (none) -> lower=0.0959931 upper=1.85005 effort=20 velocity=100; type continuous -> revolute
- joint r_wrist_pitch: limit lower=-0.436332 upper=0.436332 effort=0.65 velocity=100 -> lower=-1.13446 upper=0.174533 effort=0.65 velocity=100
- joint r_wrist_prosup: limit (none) -> lower=-0.872665 upper=0.872665 effort=0.45 velocity=100; type continuous -> revolute
- joint r_wrist_yaw: limit (none) -> lower=-0.436332 upper=0.436332 effort=0.65 velocity=100; type continuous -> revolute

File: generated/gazebo_models/iCubGenova03/icub_simulation.urdf (robot description, URDF)
Before this commit: robot test_icub, 46 links, 45 joints
Joints:
- joint l_elbow: limit (none) -> lower=0.0959931 upper=1.85005 effort=20 velocity=100; type continuous -> revolute
- joint l_wrist_pitch: limit lower=-0.436332 upper=0.436332 effort=0.65 velocity=100 -> lower=-1.13446 upper=0.174533 effort=0.65 velocity=100
- joint l_wrist_prosup: limit (none) -> lower=-0.872665 upper=0.872665 effort=0.45 velocity=100; type continuous -> revolute
- joint l_wrist_yaw: limit (none) -> lower=-0.436332 upper=0.436332 effort=0.65 velocity=100; type continuous -> revolute
- joint r_elbow: limit (none) -> lower=0.0959931 upper=1.85005 effort=20 velocity=100; type continuous -> revolute
- joint r_wrist_pitch: limit lower=-0.436332 upper=0.436332 effort=0.65 velocity=100 -> lower=-1.13446 upper=0.174533 effort=0.65 velocity=100
- joint r_wrist_prosup: limit (none) -> lower=-0.872665 upper=0.872665 effort=0.45 velocity=100; type continuous -> revolute
- joint r_wrist_yaw: limit (none) -> lower=-0.436332 upper=0.436332 effort=0.65 velocity=100; type continuous -> revolute

File: generated/urdf/iCubGenova01/icub.urdf (robot description, URDF)
Before this commit: robot test_icub, 46 links, 45 joints
Joints:
- joint l_elbow: limit (none) -> lower=0.0959931 upper=1.85005 effort=20 velocity=100; type continuous -> revolute
- joint l_wrist_pitch: limit lower=-0.436332 upper=0.436332 effort=0.65 velocity=100 -> lower=-1.13446 upper=0.174533 effort=0.65 velocity=100
- joint l_wrist_prosup: limit (none) -> lower=-0.872665 upper=0.872665 effort=0.45 velocity=100; type continuous -> revolute
- joint l_wrist_yaw: limit (none) -> lower=-0.436332 upper=0.436332 effort=0.65 velocity=100; type continuous -> revolute
- joint r_elbow: limit (none) -> lower=0.0959931 upper=1.85005 effort=20 velocity=100; type continuous -> revolute
- joint r_wrist_pitch: limit lower=-0.436332 upper=0.436332 effort=0.65 velocity=100 -> lower=-1.13446 upper=0.174533 effort=0.65 velocity=100
- joint r_wrist_prosup: limit (none) -> lower=-0.872665 upper=0.872665 effort=0.45 velocity=100; type continuous -> revolute
- joint r_wrist_yaw: limit (none) -> lower=-0.436332 upper=0.436332 effort=0.65 velocity=100; type continuous -> revolute

File: generated/urdf/iCubGenova03/icub.urdf (robot description, URDF)
Before this commit: robot test_icub, 46 links, 45 joints
Joints:
- joint l_elbow: limit (none) -> lower=0.0959931 upper=1.85005 effort=20 velocity=100; type continuous -> revolute
- joint l_wrist_pitch: limit lower=-0.436332 upper=0.436332 effort=0.65 velocity=100 -> lower=-1.13446 upper=0.174533 effort=0.65 velocity=100
- joint l_wrist_prosup: limit (none) -> lower=-0.872665 upper=0.872665 effort=0.45 velocity=100; type continuous -> revolute
- joint l_wrist_yaw: limit (none) -> lower=-0.436332 upper=0.436332 effort=0.65 velocity=100; type continuous -> revolute
- joint r_elbow: limit (none) -> lower=0.0959931 upper=1.85005 effort=20 velocity=100; type continuous -> revolute
- joint r_wrist_pitch: limit lower=-0.436332 upper=0.436332 effort=0.65 velocity=100 -> lower=-1.13446 upper=0.174533 effort=0.65 velocity=100
- joint r_wrist_prosup: limit (none) -> lower=-0.872665 upper=0.872665 effort=0.45 velocity=100; type continuous -> revolute
- joint r_wrist_yaw: limit (none) -> lower=-0.436332 upper=0.436332 effort=0.65 velocity=100; type continuous -> revolute

Commit message: cleanup of urdf_utils file

File: generated/gazebo_models/iCubGenova01/icub_simulation.urdf (robot description, URDF)
Before this commit: robot test_icub, 46 links, 45 joints
Links:
- link root_link: mass 1.2 -> 4.72

File: generated/gazebo_models/iCubGenova03/icub_simulation.urdf (robot description, URDF)
Before this commit: robot test_icub, 46 links, 45 joints
Links:
- link l_foot: mass 0.1 -> 0.761
- link r_foot: mass 0.1 -> 0.761
- link root_link: mass 1.2 -> 4.72
Joints:
- joint l_foot_ft_sensor: origin xyz=0 0 0.041 rpy=0 1.5708 0 -> xyz=-0.0035 0 0.0685 rpy=0 1.5708 0
- joint r_foot_ft_sensor: origin xyz=0 0 0.041 rpy=0 1.5708 0 -> xyz=-0.0035 4.28626e-19 0.0685 rpy=0 1.5708 0

File: generated/urdf/iCubGenova01/icub.urdf (robot description, URDF)
Before this commit: robot test_icub, 46 links, 45 joints
Links:
- removed link chest
- removed link head
- removed link imu_frame
- removed link l_ankle_1
- removed link l_arm
- removed link l_elbow_1
- removed link l_foot
- removed link l_forearm
- removed link l_gripper
- removed link l_hand
- removed link l_hip_1
- removed link l_hip_2
- removed link l_hip_3
- removed link l_shank
- removed link l_shoulder_1
- removed link l_shoulder_2
- removed link l_sole
- removed link l_thigh
- removed link l_upper_arm
- removed link l_upper_foot
- removed link l_wrist_1
- removed link lap_belt_2
- removed link neck_1
- removed link neck_2
- removed link r_ankle_1
- removed link r_arm
- removed link r_elbow_1
- removed link r_foot
- removed link r_forearm
- removed link r_gripper
- removed link r_hand
- removed link r_hip_1
- removed link r_hip_2
- removed link r_hip_3
- removed link r_shank
- removed link r_shoulder_1
- removed link r_shoulder_2
- removed link r_sole
- removed link r_thigh
- removed link r_upper_arm
- removed link r_upper_foot
- removed link r_wrist_1
- removed link torso
- link lap_belt_1: mass 0 -> 10.0; geometry 
- link root_link: mass 1.2 -> 4.72; geometry 
Joints:
- removed joint imu_frame_fixed_joint
- removed joint l_ankle_pitch
- removed joint l_ankle_roll
- removed joint l_arm_ft_sensor
- removed joint l_elbow
- removed joint l_foot_ft_sensor
- removed joint l_gripper_joint
- removed joint l_hip_pitch
- removed joint l_hip_roll
- removed joint l_hip_yaw
- removed joint l_knee
- removed joint l_leg_ft_sensor
- removed joint l_shoulder_pitch
- removed joint l_shoulder_roll
- removed joint l_shoulder_yaw
- removed joint l_sole_joint
- removed joint l_wrist_pitch
- removed joint l_wrist_prosup
- removed joint l_wrist_yaw
- removed joint neck_pitch
- removed joint neck_roll
- removed joint neck_yaw
- removed joint r_ankle_pitch
- removed joint r_ankle_roll
- removed joint r_arm_ft_sensor
- removed joint r_elbow
- removed joint r_foot_ft_sensor
- removed joint r_gripper_joint
- removed joint r_hip_pitch
- removed joint r_hip_roll
- removed joint r_hip_yaw
- removed joint r_knee
- removed joint r_leg_ft_sensor
- removed joint r_shoulder_pitch
- removed joint r_shoulder_roll
- removed joint r_shoulder_yaw
- removed joint r_sole_joint
- removed joint r_wrist_pitch
- removed joint r_wrist_prosup
- removed joint r_wrist_yaw
- removed joint torso_joint
- removed joint torso_roll
- removed joint torso_yaw
- joint torso_pitch: limit lower=-0.383972 upper=1.46608 effort=36 velocity=100 -> (none)
