Commit message: Fix joint limits (hip roll, ankle pitch) for iCubGenova03 sdf and urdf models

File: generated/gazebo_models/iCubGenova03/iCubGenova03_simulation.urdf (robot description, URDF)
Before this commit: robot test_icub, 46 links, 45 joints
Joints:
- joint l_ankle_pitch: limit lower=-0.733038 upper=0.366519 effort=24 velocity=100 -> lower=-0.4490658504 upper=0.8679448709 effort=24 velocity=100
- joint l_hip_roll: limit lower=-2.07694 upper=0.296706 effort=84 velocity=100 -> lower=-0.34 upper=1.6707963268 effort=84 velocity=100
- joint r_ankle_pitch: limit lower=-0.733038 upper=0.366519 effort=24 velocity=100 -> lower=-0.4490658504 upper=0.8679448709 effort=24 velocity=100
- joint r_hip_roll: limit lower=-2.07694 upper=0.296706 effort=84 velocity=100 -> lower=-0.34 upper=1.6707963268 effort=84 velocity=100
