Commit message: more fixes to the ankles exportation system

File: generated/gazebo_models/iCubGenova03/icub_simulation.urdf (robot description, URDF)
Before this commit: robot test_icub, 55 links, 54 joints
Joints:
- joint codyco_balancing_world_fixed_joint: origin xyz=-0.0353 -1.38778e-17 -0.001 rpy=3.14159 -0 0 -> xyz=-0.0353 -7.60894e-35 -0.001 rpy=3.14159 -0 0
- joint l_foot_ft_sensor: origin xyz=0.0135 0 0.0695 rpy=0 -0 0 -> xyz=0.017 0 0.042 rpy=0 -0 0
- joint l_sole_fixed_joint: origin xyz=-0.0353 -1.38778e-17 -0.001 rpy=3.14159 -0 0 -> xyz=-0.0353 -7.60894e-35 -0.001 rpy=3.14159 -0 0
- joint r_foot_ft_sensor: origin xyz=0.0135 4.28626e-19 0.0695 rpy=0 -0 0 -> xyz=0.017 0 0.042 rpy=0 -0 0

File: generated/gazebo_models/iCubParis01/icub_simulation.urdf (robot description, URDF)
Before this commit: robot test_icub, 55 links, 54 joints
Joints:
- joint codyco_balancing_world_fixed_joint: origin xyz=-0.0353 -1.38778e-17 -0.001 rpy=3.14159 -0 0 -> xyz=-0.0353 -7.60894e-35 -0.001 rpy=3.14159 -0 0
- joint l_foot_ft_sensor: origin xyz=0.0135 0 0.0695 rpy=0 -0 0 -> xyz=0.017 0 0.042 rpy=0 -0 0
- joint l_sole_fixed_joint: origin xyz=-0.0353 -1.38778e-17 -0.001 rpy=3.14159 -0 0 -> xyz=-0.0353 -7.60894e-35 -0.001 rpy=3.14159 -0 0
- joint r_foot_ft_sensor: origin xyz=0.0135 4.28626e-19 0.0695 rpy=0 -0 0 -> xyz=0.017 0 0.042 rpy=0 -0 0

File: generated/gazebo_models/iCubParis02/icub_simulation.urdf (robot description, URDF)
Before this commit: robot test_icub, 55 links, 54 joints
Joints:
- joint codyco_balancing_world_fixed_joint: origin xyz=-0.0353 -1.38778e-17 -0.001 rpy=3.14159 -0 0 -> xyz=-0.0263 -5.66898e-35 -0.0143 rpy=3.14159 -0 0
- joint l_foot_dh_frame_fixed_joint: origin xyz=-0.0353 0 -0.001 rpy=0 1.5708 0 -> xyz=-0.0263 0 -0.0143 rpy=0 1.5708 0
- joint l_foot_ft_sensor: origin xyz=0.0135 0 0.0695 rpy=0 -0 0 -> xyz=0.008 0 0.0553 rpy=0 -0 0
- joint l_sole_fixed_joint: origin xyz=-0.0353 -1.38778e-17 -0.001 rpy=3.14159 -0 0 -> xyz=-0.0263 -5.66898e-35 -0.0143 rpy=3.14159 -0 0
- joint r_foot_dh_frame_fixed_joint: origin xyz=-0.0353 0 -0.001 rpy=0 1.5708 0 -> xyz=-0.0263 0 -0.0143 rpy=0 1.5708 0
- joint r_foot_ft_sensor: origin xyz=0.0135 4.28626e-19 0.0695 rpy=0 -0 0 -> xyz=0.008 0 0.0553 rpy=0 -0 0
- joint r_sole_fixed_joint: origin xyz=-0.0353 -1.38778e-17 -0.001 rpy=3.14159 -0 0 -> xyz=-0.0263 -1.38778e-17 -0.0143 rpy=3.14159 -0 0

File: generated/gazebo_models/icubGazeboSim/icub_simulation.urdf (robot description, URDF)
Before this commit: robot test_icub, 55 links, 54 joints
Joints:
- joint codyco_balancing_world_fixed_joint: origin xyz=-0.0353 -1.38778e-17 -0.001 rpy=3.14159 -0 0 -> xyz=-1.24246e-32 -2.65687e-65 0.004 rpy=3.14159 -0 0
- joint l_foot_dh_frame_fixed_joint: origin xyz=-0.0353 0 -0.001 rpy=0 1.5708 0 -> xyz=0 0 0.004 rpy=0 1.5708 0
- joint l_foot_ft_sensor: origin xyz=0.0135 0 0.0695 rpy=0 -0 0 -> xyz=0 0 0.037 rpy=0 -0 0
- joint l_sole_fixed_joint: origin xyz=-0.0353 -1.38778e-17 -0.001 rpy=3.14159 -0 0 -> xyz=-1.24246e-32 -2.65687e-65 0.004 rpy=3.14159 -0 0
- joint r_foot_dh_frame_fixed_joint: origin xyz=-0.0353 0 -0.001 rpy=0 1.5708 0 -> xyz=0 0 0.004 rpy=0 1.5708 0
- joint r_foot_ft_sensor: origin xyz=0.0135 4.28626e-19 0.0695 rpy=0 -0 0 -> xyz=0 0 0.037 rpy=0 -0 0
- joint r_sole_fixed_joint: origin xyz=-0.0353 -1.38778e-17 -0.001 rpy=3.14159 -0 0 -> xyz=-1.24246e-32 -9.86076e-35 0.004 rpy=3.14159 -0 0

File: generated/urdf/iCubGenova03/icub.urdf (robot description, URDF)
Before this commit: robot test_icub, 55 links, 54 joints
Joints:
- joint codyco_balancing_world_fixed_joint: origin xyz=-0.0353 -1.38778e-17 -0.001 rpy=3.14159 -0 0 -> xyz=-0.0353 -7.60894e-35 -0.001 rpy=3.14159 -0 0
- joint l_foot_ft_sensor: origin xyz=0.0135 0 0.0695 rpy=0 -0 0 -> xyz=0.017 0 0.042 rpy=0 -0 0
- joint l_sole_fixed_joint: origin xyz=-0.0353 -1.38778e-17 -0.001 rpy=3.14159 -0 0 -> xyz=-0.0353 -7.60894e-35 -0.001 rpy=3.14159 -0 0
- joint r_foot_ft_sensor: origin xyz=0.0135 4.28626e-19 0.0695 rpy=0 -0 0 -> xyz=0.017 0 0.042 rpy=0 -0 0

File: generated/urdf/iCubParis01/icub.urdf (robot description, URDF)
Before this commit: robot test_icub, 55 links, 54 joints
Joints:
- joint codyco_balancing_world_fixed_joint: origin xyz=-0.0353 -1.38778e-17 -0.001 rpy=3.14159 -0 0 -> xyz=-0.0353 -7.60894e-35 -0.001 rpy=3.14159 -0 0
- joint l_foot_ft_sensor: origin xyz=0.0135 0 0.0695 rpy=0 -0 0 -> xyz=0.017 0 0.042 rpy=0 -0 0
- joint l_sole_fixed_joint: origin xyz=-0.0353 -1.38778e-17 -0.001 rpy=3.14159 -0 0 -> xyz=-0.0353 -7.60894e-35 -0.001 rpy=3.14159 -0 0
- joint r_foot_ft_sensor: origin xyz=0.0135 4.28626e-19 0.0695 rpy=0 -0 0 -> xyz=0.017 0 0.042 rpy=0 -0 0

File: generated/urdf/icubGazeboSim/icub.urdf (robot description, URDF)
Before this commit: robot test_icub, 55 links, 54 joints
Joints:
- joint codyco_balancing_world_fixed_joint: origin xyz=-0.0353 -1.38778e-17 -0.001 rpy=3.14159 -0 0 -> xyz=-1.24246e-32 -2.65687e-65 0.004 rpy=3.14159 -0 0
- joint l_foot_dh_frame_fixed_joint: origin xyz=-0.0353 0 -0.001 rpy=0 1.5708 0 -> xyz=0 0 0.004 rpy=0 1.5708 0
- joint l_foot_ft_sensor: origin xyz=0.0135 0 0.0695 rpy=0 -0 0 -> xyz=0 0 0.037 rpy=0 -0 0
- joint l_sole_fixed_joint: origin xyz=-0.0353 -1.38778e-17 -0.001 rpy=3.14159 -0 0 -> xyz=-1.24246e-32 -2.65687e-65 0.004 rpy=3.14159 -0 0
- joint r_foot_dh_frame_fixed_joint: origin xyz=-0.0353 0 -0.001 rpy=0 1.5708 0 -> xyz=0 0 0.004 rpy=0 1.5708 0
- joint r_foot_ft_sensor: origin xyz=0.0135 4.28626e-19 0.0695 rpy=0 -0 0 -> xyz=0 0 0.037 rpy=0 -0 0
- joint r_sole_fixed_joint: origin xyz=-0.0353 -1.38778e-17 -0.001 rpy=3.14159 -0 0 -> xyz=-1.24246e-32 -9.86076e-35 0.004 rpy=3.14159 -0 0
