Commit message: pushed new generated models

File: generated/urdf/iCubGenova01/icub.urdf (robot description, URDF)
Before this commit: robot test_two_links, 3 links, 2 joints
Links:
- added link chest, mass 4.81; collision mesh filename=meshes/collision/icub_simple_collision_chest.dae scale=1 1 1; visual mesh filename=meshes/visual/icub_chest.dae scale=1 1 1
- added link head, mass 1.33687; collision mesh filename=meshes/collision/icub_simple_collision_head.dae scale=1 1 1; visual mesh filename=meshes/visual/icub_head.dae scale=1 1 1
- added link imu_frame, mass 0
- added link l_ankle_1, mass 0.643; collision mesh filename=meshes/collision/icub_simple_collision_l_ankle_1.dae scale=1 1 1; visual mesh filename=meshes/visual/icub_l_ankle_1.dae scale=1 1 1
- added link l_arm, mass 0.727843; collision mesh filename=meshes/collision/icub_simple_collision_l_arm.dae scale=1 1 1; visual mesh filename=meshes/visual/icub_l_arm.dae scale=1 1 1
- added link l_elbow_1, mass 0.074
- added link l_foot, mass 0.761; collision mesh filename=meshes/collision/icub_simple_collision_l_foot.dae scale=1 1 1; visual mesh filename=meshes/visual/icub_l_foot.dae scale=1 1 1
- added link l_forearm, mass 0.525; collision mesh filename=meshes/collision/icub_simple_collision_l_forearm.dae scale=1 1 1; visual mesh filename=meshes/visual/icub_l_forearm.dae scale=1 1 1
- added link l_gripper, mass 0
- added link l_hand, mass 0.213; collision mesh filename=meshes/collision/icub_simple_collision_l_hand.dae scale=1 1 1; visual mesh filename=meshes/visual/icub_l_hand.dae scale=1 1 1
- added link l_hip_1, mass 0.695; collision mesh filename=meshes/collision/icub_simple_collision_l_hip_1.dae scale=1 1 1; visual mesh filename=meshes/visual/icub_l_hip_1.dae scale=1 1 1
- added link l_hip_2, mass 0.982; collision mesh filename=meshes/collision/icub_simple_collision_l_hip_2.dae scale=1 1 1; visual mesh filename=meshes/visual/icub_l_hip_2.dae scale=1 1 1
- added link l_hip_3, mass 0
- added link l_shank, mass 2.032; collision mesh filename=meshes/collision/icub_simple_collision_l_shank.dae scale=1 1 1; visual mesh filename=meshes/visual/icub_l_shank.dae scale=1 1 1
- added link l_shoulder_1, mass 0.189; collision mesh filename=meshes/collision/icub_simple_collision_l_shoulder_1.dae scale=1 1 1; visual mesh filename=meshes/visual/icub_l_shoulder_1.dae scale=1 1 1
- added link l_shoulder_2, mass 0.179; collision mesh filename=meshes/collision/icub_simple_collision_l_shoulder_2.dae scale=1 1 1; visual mesh filename=meshes/visual/icub_l_shoulder_2.dae scale=1 1 1
- added link l_sole, mass 0
- added link l_thigh, mass 1.522; collision mesh filename=meshes/collision/icub_simple_collision_l_thigh.dae scale=1 1 1; visual mesh filename=meshes/visual/icub_l_thigh.dae scale=1 1 1
- added link l_upper_arm, mass 0.156157
- added link l_upper_foot, mass 0.1
- added link l_wrist_1, mass 0
- added link lap_belt_2, mass 0
- added link neck_1, mass 0; collision mesh filename=meshes/collision/icub_simple_collision_neck_1.dae scale=1 1 1; visual mesh filename=meshes/visual/icub_neck_1.dae scale=1 1 1
- added link neck_2, mass 0; collision mesh filename=meshes/collision/icub_simple_collision_neck_2.dae scale=1 1 1; visual mesh filename=meshes/visual/icub_neck_2.dae scale=1 1 1
- added link r_ankle_1, mass 0.643; collision mesh filename=meshes/collision/icub_simple_collision_r_ankle_1.dae scale=1 1 1; visual mesh filename=meshes/visual/icub_r_ankle_1.dae scale=1 1 1
- added link r_arm, mass 0.729; collision mesh filename=meshes/collision/icub_simple_collision_r_arm.dae scale=1 1 1; visual mesh filename=meshes/visual/icub_r_arm.dae scale=1 1 1
- added link r_elbow_1, mass 0.074
- added link r_foot, mass 0.761; collision mesh filename=meshes/collision/icub_simple_collision_r_foot.dae scale=1 1 1; visual mesh filename=meshes/visual/icub_r_foot.dae scale=1 1 1
- added link r_forearm, mass 0.525; collision mesh filename=meshes/collision/icub_simple_collision_r_forearm.dae scale=1 1 1; visual mesh filename=meshes/visual/icub_r_forearm.dae scale=1 1 1
- added link r_gripper, mass 0
- added link r_hand, mass 0.213; collision mesh filename=meshes/collision/icub_simple_collision_r_hand.dae scale=1 1 1; visual mesh filename=meshes/visual/icub_r_hand.dae scale=1 1 1
- added link r_hip_1, mass 0.695; collision mesh filename=meshes/collision/icub_simple_collision_r_hip_1.dae scale=1 1 1; visual mesh filename=meshes/visual/icub_r_hip_1.dae scale=1 1 1
- added link r_hip_2, mass 0.982; collision mesh filename=meshes/collision/icub_simple_collision_r_hip_2.dae scale=1 1 1; visual mesh filename=meshes/visual/icub_r_hip_2.dae scale=1 1 1
- added link r_hip_3, mass 0
- added link r_shank, mass 2.032; collision mesh filename=meshes/collision/icub_simple_collision_r_shank.dae scale=1 1 1; visual mesh filename=meshes/visual/icub_r_shank.dae scale=1 1 1
- added link r_shoulder_1, mass 0.189; collision mesh filename=meshes/collision/icub_simple_collision_r_shoulder_1.dae scale=1 1 1; visual mesh filename=meshes/visual/icub_r_shoulder_1.dae scale=1 1 1
- added link r_shoulder_2, mass 0.179; collision mesh filename=meshes/collision/icub_simple_collision_r_shoulder_2.dae scale=1 1 1; visual mesh filename=meshes/visual/icub_r_shoulder_2.dae scale=1 1 1
- added link r_sole, mass 0
- added link r_thigh, mass 1.522; collision mesh filename=meshes/collision/icub_simple_collision_r_thigh.dae scale=1 1 1; visual mesh filename=meshes/visual/icub_r_thigh.dae scale=1 1 1
- added link r_upper_arm, mass 0.155
- added link r_upper_foot, mass 0.1
- added link r_wrist_1, mass 0
- added link torso, mass 0
- link lap_belt_1: mass 10.0 -> 0; geometry collision mesh filename=meshes/collision/icub_simple_collision_lap_belt_1.dae scale=1 1 1; visual mesh filename=meshes/visual/icub_lap_belt_1.dae scale=1 1 1
- link root_link: geometry collision mesh filename=meshes/collision/icub_simple_collision_root_link.dae scale=1 1 1; visual mesh filename=meshes/visual/icub_root_link.dae scale=1 1 1
Joints:
- added joint imu_frame_fixed_joint: type fixed, parent head, child imu_frame, origin xyz=0.0185 -0.1108 0.0066 rpy=1.5708 -0 0, axis 0 0 0
- added joint l_ankle_pitch: type revolute, parent l_shank, child l_ankle_1, origin xyz=-0.2005 0 0 rpy=-1.5708 0 0, axis 0 -1 6.12323e-17, limit lower=-0.733038 upper=0.366519 effort=24 velocity=100
- added joint l_ankle_roll: type revolute, parent l_ankle_1, child l_upper_foot, origin xyz=0 0 0 rpy=0 -1.5708 0, axis 1 0 0, limit lower=-0.418879 upper=0.418879 effort=11 velocity=100
- added joint l_arm_ft_sensor: type fixed, parent l_upper_arm, child l_arm, origin xyz=0.015 9.36797e-18 0.15228 rpy=-1.5708 0 0, axis 0 0 0
- added joint l_elbow: type revolute, parent l_arm, child l_elbow_1, origin xyz=0 0 0 rpy=1.5708 -0 0, axis 0 1 6.12323e-17, limit lower=0.0959931 upper=1.85005 effort=20 velocity=100
- added joint l_foot_ft_sensor: type fixed, parent l_upper_foot, child l_foot, origin xyz=-0.0035 0 0.0685 rpy=0 1.5708 0, axis 0 0 0
- added joint l_gripper_joint: type fixed, parent l_hand, child l_gripper, origin xyz=0.0625 0 -0.016 rpy=0 -0 0, axis 0 0 0
- added joint l_hip_pitch: type revolute, parent root_link, child l_hip_1, origin xyz=0 -0.0681 -0.1199 rpy=-3.14159 1.5708 -2.77556e-17, axis 0 -1 6.12323e-17, limit lower=-0.767945 upper=2.30383 effort=84 velocity=100
- added joint l_hip_roll: type revolute, parent l_hip_1, child l_hip_2, origin xyz=0 0 0 rpy=3.14159 -1.5708 -2.77556e-17, axis 1 0 -6.12323e-17, limit lower=-2.07694 upper=0.296706 effort=84 velocity=100
- added joint l_hip_yaw: type revolute, parent l_hip_3, child l_thigh, origin xyz=1.68519e-34 0 0 rpy=1.5708 -0 -1.5708, axis 0 1 6.12323e-17, limit lower=-1.37881 upper=1.37881 effort=40 velocity=100
- added joint l_knee: type revolute, parent l_thigh, child l_shank, origin xyz=-0.0009175 -0.234545 -1.43617e-17 rpy=3.14159 -1.2326e-32 1.5708, axis 0 1.22465e-16 -1, limit lower=-2.18166 upper=0.401426 effort=30 velocity=100
- added joint l_leg_ft_sensor: type fixed, parent l_hip_2, child l_hip_3, origin xyz=0 0 0 rpy=3.14159 0 -1.5708, axis 0 0 0
- added joint l_shoulder_pitch: type revolute, parent chest, child l_shoulder_1, origin xyz=0.00525 0.1433 -0.11026 rpy=1.309 5.55112e-17 1.5708, axis 0 -1 5.55112e-17, limit lower=-1.65806 upper=0.0872665 effort=84 velocity=100
- added joint l_shoulder_roll: type revolute, parent l_shoulder_1, child l_shoulder_2, origin xyz=0 0 0 rpy=1.5708 -0 -1.5708, axis 0 1 6.12323e-17, limit lower=0 upper=2.80649 effort=84 velocity=100
- added joint l_shoulder_yaw: type revolute, parent l_shoulder_2, child l_upper_arm, origin xyz=4.33681e-19 1.73472e-18 0 rpy=6.12323e-17 -0 1.309, axis 0 6.12323e-17 1, limit lower=-0.645772 upper=1.74533 effort=34 velocity=100
- added joint l_sole_joint: type fixed, parent l_foot, child l_sole, origin xyz=0 0 0 rpy=0 -0 0, axis 0 0 0
- added joint l_wrist_pitch: type revolute, parent l_forearm, child l_wrist_1, origin xyz=0 0.1373 8.4072e-18 rpy=1.5708 -0 1.5708, axis 0 1 6.12323e-17, limit lower=-1.13446 upper=0.174533 effort=0.65 velocity=100
- added joint l_wrist_prosup: type revolute, parent l_elbow_1, child l_forearm, origin xyz=-0.015 0 0 rpy=1.5708 -0 -1.5708, axis 0 1 6.12323e-17, limit lower=-0.872665 upper=0.872665 effort=0.45 velocity=100
- added joint l_wrist_yaw: type revolute, parent l_wrist_1, child l_hand, origin xyz=0 0 0 rpy=0 -0 0, axis 0 0 1, limit lower=-0.436332 upper=0.436332 effort=0.65 velocity=100
- added joint neck_pitch: type revolute, parent chest, child neck_1, origin xyz=0.00231 0.1933 -1.18362e-17 rpy=1.5708 -0 1.5708, axis 0 1 6.12323e-17, limit lower=-0.698132 upper=0.523599 effort=20 velocity=100
- added joint neck_roll: type revolute, parent neck_1, child neck_2, origin xyz=0.0095 0 0 rpy=-1.5708 -0 -1.5708, axis 0 -1 6.12323e-17, limit lower=-1.22173 upper=1.0472 effort=20 velocity=100
- added joint neck_yaw: type revolute, parent neck_2, child head, origin xyz=-5.77779e-34 0 0 rpy=-1.5708 -0 1.5708, axis 0 -1 6.12323e-17, limit lower=-0.959931 upper=0.959931 effort=20 velocity=100
- added joint r_ankle_pitch: type revolute, parent r_shank, child r_ankle_1, origin xyz=-0.2005 0 0 rpy=1.5708 -0 0, axis 0 1 6.12323e-17, limit lower=-0.733038 upper=0.366519 effort=24 velocity=100
- added joint r_ankle_roll: type revolute, parent r_ankle_1, child r_upper_foot, origin xyz=0 0 0 rpy=0.504019 1.5708 -2.63757, axis -1 1.22465e-16 0, limit lower=-0.418879 upper=0.418879 effort=11 velocity=100
- added joint r_arm_ft_sensor: type fixed, parent r_upper_arm, child r_arm, origin xyz=0.015 -8.93429e-18 0.15228 rpy=1.5708 -0 3.14159, axis 0 0 0
- added joint r_elbow: type revolute, parent r_arm, child r_elbow_1, origin xyz=0 0 0 rpy=1.5708 -0 0, axis 0 1 6.12323e-17, limit lower=0.0959931 upper=1.85005 effort=20 velocity=100
- added joint r_foot_ft_sensor: type fixed, parent r_upper_foot, child r_foot, origin xyz=-0.0035 4.28626e-19 0.0685 rpy=0 1.5708 0, axis 0 0 0
- added joint r_gripper_joint: type fixed, parent r_hand, child r_gripper, origin xyz=0.0625 0 0.016 rpy=0 -0 0, axis 0 0 0
- added joint r_hip_pitch: type revolute, parent root_link, child r_hip_1, origin xyz=0 0.0681 -0.1199 rpy=-2.77556e-17 1.5708 2.77556e-17, axis 0 1 6.12323e-17, limit lower=-0.767945 upper=2.30383 effort=84 velocity=100
- added joint r_hip_roll: type revolute, parent r_hip_1, child r_hip_2, origin xyz=0 0 0 rpy=2.77556e-17 1.5708 -2.77556e-17, axis -1 0 6.12323e-17, limit lower=-2.07694 upper=0.296706 effort=84 velocity=100
- added joint r_hip_yaw: type revolute, parent r_hip_3, child r_thigh, origin xyz=1.68519e-34 0 0 rpy=-1.5708 -0 -1.5708, axis 0 -1 6.12323e-17, limit lower=-1.37881 upper=1.37881 effort=40 velocity=100
- added joint r_knee: type revolute, parent r_thigh, child r_shank, origin xyz=-0.0009175 -0.234545 1.43617e-17 rpy=3.14159 -1.2326e-32 1.5708, axis 0 1.22465e-16 -1, limit lower=-2.18166 upper=0.401426 effort=30 velocity=100
- added joint r_leg_ft_sensor: type fixed, parent r_hip_2, child r_hip_3, origin xyz=0 0 0 rpy=0 -0 1.5708, axis 0 0 0
- added joint r_shoulder_pitch: type revolute, parent chest, child r_shoulder_1, origin xyz=0.00525 0.1433 0.11026 rpy=-1.309 -0 1.5708, axis 0 1 5.55112e-17, limit lower=-1.65806 upper=0.0872665 effort=84 velocity=100
- added joint r_shoulder_roll: type revolute, parent r_shoulder_1, child r_shoulder_2, origin xyz=0 0 0 rpy=-1.5708 -0 -1.5708, axis 0 -1 6.12323e-17, limit lower=0 upper=2.80649 effort=84 velocity=100
- added joint r_shoulder_yaw: type revolute, parent r_shoulder_2, child r_upper_arm, origin xyz=-4.33681e-19 0 0 rpy=3.14159 -0 1.309, axis 0 6.12323e-17 -1, limit lower=-0.645772 upper=1.74533 effort=34 velocity=100
- added joint r_sole_joint: type fixed, parent r_foot, child r_sole, origin xyz=0 0 0 rpy=0 -0 0, axis 0 0 0
- added joint r_wrist_pitch: type revolute, parent r_forearm, child r_wrist_1, origin xyz=0 -0.1373 -8.4072e-18 rpy=1.5708 -0 1.5708, axis 0 1 6.12323e-17, limit lower=-1.13446 upper=0.174533 effort=0.65 velocity=100
- added joint r_wrist_prosup: type revolute, parent r_elbow_1, child r_forearm, origin xyz=0.015 0 0 rpy=1.5708 -0 -1.5708, axis 0 1 6.12323e-17, limit lower=-0.872665 upper=0.872665 effort=0.45 velocity=100
- added joint r_wrist_yaw: type revolute, parent r_wrist_1, child r_hand, origin xyz=0 0 0 rpy=0 -0 3.14159, axis 0 0 1, limit lower=-0.436332 upper=0.436332 effort=0.65 velocity=100
- added joint torso_joint: type fixed, parent chest, child torso, origin xyz=0.00231 0.1933 -1.18362e-17 rpy=0 -0 0, axis 0 0 0
- added joint torso_roll: type revolute, parent lap_belt_1, child lap_belt_2, origin xyz=0.032 -2.67276e-51 0 rpy=1.5708 -0 -1.5708, axis 0 1 6.12323e-17, limit lower=-0.680678 upper=0.680678 effort=80 velocity=100
- added joint torso_yaw: type revolute, parent lap_belt_2, child chest, origin xyz=-7.46298e-34 -0.0055 0 rpy=-1.5708 -0 -1.5708, axis 0 -1 6.12323e-17, limit lower=-1.02974 upper=1.02974 effort=80 velocity=100
- joint torso_pitch: limit (none) -> lower=-0.383972 upper=1.46608 effort=36 velocity=100

Commit message: Push update iCubGenova* models

File: generated/urdf/iCubGenova01/icub.urdf (robot description, URDF)
Before this commit: robot test_icub, 46 links, 45 joints
Links:
- removed link l_shank
- removed link r_shank
- added link l_leg, mass 2.032
- added link r_leg, mass 2.032
Joints:
- joint l_ankle_pitch: parent l_shank -> l_leg
- joint l_knee: child l_shank -> l_leg
- joint r_ankle_pitch: parent r_shank -> r_leg
- joint r_knee: child r_shank -> r_leg

File: generated/urdf/iCubGenova03/icub.urdf (robot description, URDF)
Before this commit: robot test_icub, 46 links, 45 joints
Links:
- removed link l_shank
- removed link r_shank
- added link l_leg, mass 1.264
- added link r_leg, mass 1.264
Joints:
- joint l_ankle_pitch: parent l_shank -> l_leg
- joint l_knee: child l_shank -> l_leg
- joint r_ankle_pitch: parent r_shank -> r_leg
- joint r_knee: child r_shank -> r_leg

Commit message: push new generated files

File: generated/urdf/iCubGenova01/icub.urdf (robot description, URDF)
Before this commit: robot test_icub, 46 links, 45 joints
Links:
- removed link lap_belt_1
- removed link lap_belt_2
- added link torso_1, mass 0; collision mesh filename=meshes/collision/icub_simple_collision_lap_belt_1.dae scale=1 1 1; visual mesh filename=meshes/visual/icub_lap_belt_1.dae scale=1 1 1
- added link torso_2, mass 0
- link l_leg: geometry collision mesh filename=meshes/collision/icub_simple_collision_l_shank.dae scale=1 1 1; visual mesh filename=meshes/visual/icub_l_shank.dae scale=1 1 1
- link r_leg: geometry collision mesh filename=meshes/collision/icub_simple_collision_r_shank.dae scale=1 1 1; visual mesh filename=meshes/visual/icub_r_shank.dae scale=1 1 1
Joints:
- joint torso_pitch: child lap_belt_1 -> torso_1
- joint torso_roll: child lap_belt_2 -> torso_2; parent lap_belt_1 -> torso_1
- joint torso_yaw: parent lap_belt_2 -> torso_2

File: generated/urdf/iCubGenova03/icub.urdf (robot description, URDF)
Before this commit: robot test_icub, 46 links, 45 joints
Links:
- removed link lap_belt_1
- removed link lap_belt_2
- added link torso_1, mass 0; collision mesh filename=meshes/collision/icub_simple_collision_lap_belt_1.dae scale=1 1 1; visual mesh filename=meshes/visual/icub_lap_belt_1.dae scale=1 1 1
- added link torso_2, mass 0
- link l_leg: geometry collision mesh filename=meshes/collision/icub_simple_collision_l_shank.dae scale=1 1 1; visual mesh filename=meshes/visual/icub_l_shank.dae scale=1 1 1
- link r_leg: geometry collision mesh filename=meshes/collision/icub_simple_collision_r_shank.dae scale=1 1 1; visual mesh filename=meshes/visual/icub_r_shank.dae scale=1 1 1
Joints:
- joint torso_pitch: child lap_belt_1 -> torso_1
- joint torso_roll: child lap_belt_2 -> torso_2; parent lap_belt_1 -> torso_1
- joint torso_yaw: parent lap_belt_2 -> torso_2

Commit message: corrected head mass, see https://github.com/robotology/codyco-modules/issues/49

File: generated/urdf/iCubGenova01/icub.urdf (robot description, URDF)
Before this commit: robot test_icub, 46 links, 45 joints
Links:
- link head: mass 1.33687 -> 3

File: generated/urdf/iCubGenova03/icub.urdf (robot description, URDF)
Before this commit: robot test_icub, 46 links, 45 joints
Links:
- link head: mass 1.33687 -> 3
