Commit message: update models with modification for stable gazebo use

File: generated/gazebo_models/iCubParis01/icub_simulation.urdf (robot description, URDF)
Before this commit: robot test_icub, 55 links, 54 joints
Links:
- link neck_1: mass 0.1 -> 0.270176
- link neck_2: mass 0.1 -> 0.272306
Joints:
- joint imu_frame_fixed_joint: origin xyz=0.0185 -0.1108 0.0066 rpy=1.5708 -0 0 -> xyz=0.0225 -0.1005 0.0066 rpy=1.5708 -0 0
- joint neck_roll: origin xyz=0.0095 0 0 rpy=-1.5708 -0 -1.5708 -> xyz=0.033 -2.13821e-50 0 rpy=-1.5708 -0 -1.5708
- joint neck_yaw: origin xyz=-5.77779e-34 0 0 rpy=-1.5708 -0 1.5708 -> xyz=0 -0.001 0 rpy=-1.5708 -0 1.5708

File: generated/urdf/iCubParis01/icub.urdf (robot description, URDF)
Before this commit: robot test_icub, 55 links, 54 joints
Links:
- link neck_1: mass 0 -> 0.270176
- link neck_2: mass 0 -> 0.272306
Joints:
- joint imu_frame_fixed_joint: origin xyz=0.0185 -0.1108 0.0066 rpy=1.5708 -0 0 -> xyz=0.0225 -0.1005 0.0066 rpy=1.5708 -0 0
- joint neck_roll: origin xyz=0.0095 0 0 rpy=-1.5708 -0 -1.5708 -> xyz=0.033 -2.13821e-50 0 rpy=-1.5708 -0 -1.5708
- joint neck_yaw: origin xyz=-5.77779e-34 0 0 rpy=-1.5708 -0 1.5708 -> xyz=0 -0.001 0 rpy=-1.5708 -0 1.5708
