Commit message: added generation of icubGazeboSim model without ft sensors

File: generated/gazebo_models/icubGazeboSimNoFT/icub_simulation.urdf (robot description, URDF)
Before this commit: robot test_icub, 46 links, 45 joints
Links:
- removed link l_arm
- removed link l_shank
- removed link l_thigh
- removed link l_upper_foot
- removed link lap_belt_1
- removed link lap_belt_2
- removed link r_arm
- removed link r_shank
- removed link r_thigh
- removed link r_upper_foot
- added link codyco_balancing_world, mass 0
- added link l_ankle_2, mass 0.2675
- added link l_foot_dh_frame, mass 0
- added link l_forearm_dh_frame, mass 0
- added link l_hand_dh_frame, mass 0
- added link l_lower_leg, mass 1.264; collision mesh filename=meshes/collision/icub_simple_collision_l_shank.dae scale=1 1 1; visual mesh filename=meshes/visual/icub_l_shank.dae scale=1 1 1
- added link l_shoulder_3, mass 0.156157
- added link l_upper_arm_dh_frame, mass 0
- added link l_upper_leg, mass 2.175; collision mesh filename=meshes/collision/icub_simple_collision_l_thigh.dae scale=1 1 1; visual mesh filename=meshes/visual/icub_l_thigh.dae scale=1 1 1
- added link r_ankle_2, mass 0.2675
- added link r_foot_dh_frame, mass 0
- added link r_forearm_dh_frame, mass 0
- added link r_hand_dh_frame, mass 0
- added link r_lower_leg, mass 1.264; collision mesh filename=meshes/collision/icub_simple_collision_r_shank.dae scale=1 1 1; visual mesh filename=meshes/visual/icub_r_shank.dae scale=1 1 1
- added link r_shoulder_3, mass 0.155
- added link r_upper_arm_dh_frame, mass 0
- added link r_upper_leg, mass 2.175; collision mesh filename=meshes/collision/icub_simple_collision_r_thigh.dae scale=1 1 1; visual mesh filename=meshes/visual/icub_r_thigh.dae scale=1 1 1
- added link torso_1, mass 0.1; collision mesh filename=meshes/collision/icub_simple_collision_lap_belt_1.dae scale=1 1 1; visual mesh filename=meshes/visual/icub_lap_belt_1.dae scale=1 1 1
- added link torso_2, mass 0.1
- link head: mass 1.33687 -> 3
- link l_ankle_1: mass 0.643 -> 0.746
- link l_foot: mass 0.761 -> 0.5935
- link l_hip_1: mass 0.695 -> 0.754
- link l_hip_2: mass 0.982 -> 0.526
- link l_upper_arm: mass 0.156157 -> 0.727843; geometry collision mesh filename=meshes/collision/icub_simple_collision_l_arm.dae scale=1 1 1; visual mesh filename=meshes/visual/icub_l_arm.dae scale=1 1 1
- link r_ankle_1: mass 0.643 -> 0.746
- link r_foot: mass 0.761 -> 0.5935
- link r_hip_1: mass 0.695 -> 0.754
- link r_hip_2: mass 0.982 -> 0.526
- link r_upper_arm: mass 0.155 -> 0.729; geometry collision mesh filename=meshes/collision/icub_simple_collision_r_arm.dae scale=1 1 1; visual mesh filename=meshes/visual/icub_r_arm.dae scale=1 1 1
Joints:
- removed joint l_sole_joint
- removed joint r_sole_joint
- added joint codyco_balancing_world_fixed_joint: type fixed, parent l_foot, child codyco_balancing_world, origin xyz=-1.24246e-32 -2.65687e-65 0.004 rpy=3.14159 -0 0, axis 0 0 0
- added joint l_foot_dh_frame_fixed_joint: type fixed, parent l_foot, child l_foot_dh_frame, origin xyz=0 0 0.004 rpy=0 1.5708 0, axis 0 0 0
- added joint l_forearm_dh_frame_fixed_joint: type fixed, parent l_forearm, child l_forearm_dh_frame, origin xyz=0 0.1373 8.4072e-18 rpy=0 -0 0, axis 0 0 0
- added joint l_hand_dh_frame_fixed_joint: type fixed, parent l_hand, child l_hand_dh_frame, origin xyz=0.0625 0 -0.016 rpy=0 -0 0, axis 0 0 0
- added joint l_sole_fixed_joint: type fixed, parent l_foot, child l_sole, origin xyz=-1.24246e-32 -2.65687e-65 0.004 rpy=3.14159 -0 0, axis 0 0 0
- added joint l_upper_arm_dh_frame_fixed_joint: type fixed, parent l_upper_arm, child l_upper_arm_dh_frame, origin xyz=0 0 0.08428 rpy=-1.5708 0 0, axis 0 0 0
- added joint r_foot_dh_frame_fixed_joint: type fixed, parent r_foot, child r_foot_dh_frame, origin xyz=0 0 0.004 rpy=0 1.5708 0, axis 0 0 0
- added joint r_forearm_dh_frame_fixed_joint: type fixed, parent r_forearm, child r_forearm_dh_frame, origin xyz=0 -0.1373 -8.4072e-18 rpy=0 -0 0, axis 0 0 0
- added joint r_hand_dh_frame_fixed_joint: type fixed, parent r_hand, child r_hand_dh_frame, origin xyz=0.0625 0 0.016 rpy=0 -0 0, axis 0 0 0
- added joint r_sole_fixed_joint: type fixed, parent r_foot, child r_sole, origin xyz=-1.24246e-32 -9.86076e-35 0.004 rpy=3.14159 -0 0, axis 0 0 0
- added joint r_upper_arm_dh_frame_fixed_joint: type fixed, parent r_upper_arm, child r_upper_arm_dh_frame, origin xyz=0 0 0.08428 rpy=1.5708 -0 3.14159, axis 0 0 0
- joint l_ankle_pitch: origin xyz=-0.2005 0 0 rpy=-1.5708 0 0 -> xyz=-0.213 0 0 rpy=-1.5708 0 0; parent l_shank -> l_lower_leg
- joint l_ankle_roll: child l_upper_foot -> l_ankle_2
- joint l_arm_ft_sensor: child l_arm -> l_upper_arm; origin xyz=0.015 9.36797e-18 0.15228 rpy=-1.5708 0 0 -> xyz=0.015 9.36797e-18 0.068 rpy=0 -0 0; parent l_upper_arm -> l_shoulder_3
- joint l_elbow: origin xyz=0 0 0 rpy=1.5708 -0 0 -> xyz=0 0 0.08428 rpy=-6.12323e-17 0 0; parent l_arm -> l_upper_arm
- joint l_foot_ft_sensor: origin xyz=-0.0035 0 0.0685 rpy=0 1.5708 0 -> xyz=0 0 0.037 rpy=0 -0 0; parent l_upper_foot -> l_ankle_2
- joint l_hip_yaw: child l_thigh -> l_upper_leg; origin xyz=1.68519e-34 0 0 rpy=1.5708 -0 -1.5708 -> xyz=0 0 -0.0665 rpy=-1.5708 -6.16298e-33 -6.12323e-17
- joint l_knee: child l_shank -> l_lower_leg; origin xyz=-0.0009175 -0.234545 -1.43617e-17 rpy=3.14159 -1.2326e-32 1.5708 -> xyz=0 -0.2236 -1.36916e-17 rpy=3.14159 -1.2326e-32 1.5708; parent l_thigh -> l_upper_leg
- joint l_leg_ft_sensor: origin xyz=0 0 0 rpy=3.14159 0 -1.5708 -> xyz=0 0 0.0665 rpy=0 -0 0
- joint l_shoulder_yaw: child l_upper_arm -> l_shoulder_3
- joint r_ankle_pitch: origin xyz=-0.2005 0 0 rpy=1.5708 -0 0 -> xyz=-0.213 0 0 rpy=1.5708 -0 0; parent r_shank -> r_lower_leg
- joint r_ankle_roll: child r_upper_foot -> r_ankle_2
- joint r_arm_ft_sensor: child r_arm -> r_upper_arm; origin xyz=0.015 -8.93429e-18 0.15228 rpy=1.5708 -0 3.14159 -> xyz=0.015 -8.93429e-18 0.068 rpy=0 -0 0; parent r_upper_arm -> r_shoulder_3
- joint r_elbow: origin xyz=0 0 0 rpy=1.5708 -0 0 -> xyz=0 0 0.08428 rpy=3.14159 -0 3.14159; parent r_arm -> r_upper_arm
- joint r_foot_ft_sensor: origin xyz=-0.0035 4.28626e-19 0.0685 rpy=0 1.5708 0 -> xyz=0 0 0.037 rpy=0 -0 0; parent r_upper_foot -> r_ankle_2
- joint r_hip_yaw: child r_thigh -> r_upper_leg; origin xyz=1.68519e-34 0 0 rpy=-1.5708 -0 -1.5708 -> xyz=0 0 -0.0665 rpy=-1.5708 -6.16298e-33 6.12323e-17
- joint r_knee: child r_shank -> r_lower_leg; origin xyz=-0.0009175 -0.234545 1.43617e-17 rpy=3.14159 -1.2326e-32 1.5708 -> xyz=0 -0.2236 1.36916e-17 rpy=3.14159 -1.2326e-32 1.5708; parent r_thigh -> r_upper_leg
- joint r_leg_ft_sensor: origin xyz=0 0 0 rpy=0 -0 1.5708 -> xyz=0 0 0.0665 rpy=0 -0 0
- joint r_shoulder_yaw: child r_upper_arm -> r_shoulder_3
- joint torso_pitch: child lap_belt_1 -> torso_1
- joint torso_roll: child lap_belt_2 -> torso_2; parent lap_belt_1 -> torso_1
- joint torso_yaw: parent lap_belt_2 -> torso_2
