Commit message: Regenerated models after the fix of the bug in generation of the r_foot_dh_frame frame, fixed in https://github.com/robotology-playground/idyntree/commit/c6394e90e23318cc0fd726855b8ad6d3764d4e25

File: generated/gazebo_models/iCubDarmstad01/icub_simulation.urdf (robot description, URDF)
Before this commit: robot test_icub, 55 links, 54 joints
Joints:
- joint r_foot_dh_frame_fixed_joint: origin xyz=-4.29004e-17 -0.1362 0.075 rpy=-0.834365 1.5708 -0.834365 -> xyz=-8.67362e-19 1.38778e-17 0.075 rpy=-1.01315e-16 1.5708 -1.01315e-16

File: generated/gazebo_models/iCubGenova03/icub_simulation.urdf (robot description, URDF)
Before this commit: robot test_icub, 55 links, 54 joints
Joints:
- joint r_foot_dh_frame_fixed_joint: origin xyz=-4.2033e-17 -0.1362 0.075 rpy=-0.834365 1.5708 -0.834365 -> xyz=-1.84889e-33 -1.84889e-33 0.075 rpy=-1.01315e-16 1.5708 -1.01315e-16

File: generated/urdf/iCubGenova03/icub.urdf (robot description, URDF)
Before this commit: robot test_icub, 55 links, 54 joints
Joints:
- joint r_foot_dh_frame_fixed_joint: origin xyz=-4.2033e-17 -0.1362 0.075 rpy=-0.834365 1.5708 -0.834365 -> xyz=-1.84889e-33 -1.84889e-33 0.075 rpy=-1.01315e-16 1.5708 -1.01315e-16
