Commit message: Commit generated models

File: generated/robots/iCubDarmstadt01/model.urdf (robot description, URDF)
Before this commit: robot ICUB_2-5_BB_SIM_MODEL, 104 links, 103 joints
Links:
- added link l_foot_dh_frame
- added link r_foot_dh_frame
Joints:
- added joint l_foot_dh_frame_fixed_joint: type fixed, parent l_foot, child l_foot_dh_frame, origin xyz=0.0 0 0.004 rpy=0 1.5708 0, axis 0 0 0
- added joint r_foot_dh_frame_fixed_joint: type fixed, parent r_foot, child r_foot_dh_frame, origin xyz=0.0 0 0.004 rpy=0 1.5708 0, axis 0 0 0

File: generated/robots/iCubGenova02/model.urdf (robot description, URDF)
Before this commit: robot ICUB_2-5_BB_SIM_MODEL, 104 links, 103 joints
Links:
- added link l_foot_dh_frame
- added link r_foot_dh_frame
Joints:
- added joint l_foot_dh_frame_fixed_joint: type fixed, parent l_foot, child l_foot_dh_frame, origin xyz=0.0 0 0.004 rpy=0 1.5708 0, axis 0 0 0
- added joint r_foot_dh_frame_fixed_joint: type fixed, parent r_foot, child r_foot_dh_frame, origin xyz=0.0 0 0.004 rpy=0 1.5708 0, axis 0 0 0

Commit message: added generation of iDynTree style F/T sensors

File: generated/robots/iCubDarmstadt01/model.urdf (robot description, URDF)
Before this commit: robot ICUB_2-5_BB_SIM_MODEL, 106 links, 105 joints
Joints:
- joint l_knee: axis -1.0 0.0 0.0 -> -1.0 -0.0 -0.0
- joint r_ankle_roll: axis 0.0 0.0 -1.0 -> -0.0 -0.0 -1.0
- joint r_hip_pitch: axis -1.0 0.0 0.0 -> -1.0 -0.0 -0.0
- joint r_hip_roll: axis 0.0 0.0 -1.0 -> -0.0 -0.0 -1.0

File: generated/robots/iCubGenova02/model.urdf (robot description, URDF)
Before this commit: robot ICUB_2-5_BB_SIM_MODEL, 106 links, 105 joints
Joints:
- joint l_knee: axis -1.0 0.0 0.0 -> -1.0 -0.0 -0.0
- joint r_ankle_roll: axis 0.0 0.0 -1.0 -> -0.0 -0.0 -1.0
- joint r_hip_pitch: axis -1.0 0.0 0.0 -> -1.0 -0.0 -0.0
- joint r_hip_roll: axis 0.0 0.0 -1.0 -> -0.0 -0.0 -1.0

Commit message: Regenerated the model files after the simmechanics-to-urdf script fix #21

File: generated/robots/iCubDarmstadt01/model.urdf (robot description, URDF)
Before this commit: robot ICUB_2-5_BB_SIM_MODEL, 106 links, 105 joints
Links:
- added link imu
Joints:
- added joint imu_fixed_joint: type fixed, parent head, child imu, origin xyz=0.00950000019074 0.133444 0.0093 rpy=-1.57079632679 1.57079632679 0
- joint l_knee: axis -1.0 -0.0 -0.0 -> -1.0 0.0 0.0
- joint r_ankle_roll: axis -0.0 -0.0 -1.0 -> 0.0 0.0 -1.0
- joint r_hip_pitch: axis -1.0 -0.0 -0.0 -> -1.0 0.0 0.0
- joint r_hip_roll: axis -0.0 -0.0 -1.0 -> 0.0 0.0 -1.0

File: generated/robots/iCubGenova02/model.urdf (robot description, URDF)
Before this commit: robot ICUB_2-5_BB_SIM_MODEL, 106 links, 105 joints
Links:
- added link imu
Joints:
- added joint imu_fixed_joint: type fixed, parent head, child imu, origin xyz=0.00950000019074 0.133444 0.0093 rpy=-1.57079632679 1.57079632679 0
- joint l_knee: axis -1.0 -0.0 -0.0 -> -1.0 0.0 0.0
- joint r_ankle_roll: axis -0.0 -0.0 -1.0 -> 0.0 0.0 -1.0
- joint r_hip_pitch: axis -1.0 -0.0 -0.0 -> -1.0 0.0 0.0
- joint r_hip_roll: axis -0.0 -0.0 -1.0 -> 0.0 0.0 -1.0

Commit message: Regenerated the URDF models

File: generated/robots/iCubDarmstadt01/model.urdf (robot description, URDF)
Before this commit: robot ICUB_2-5_BB_SIM_MODEL, 107 links, 106 joints
Links:
- added link l_forearm_mtb_acc_1b7
- added link l_forearm_mtb_acc_1b8
- added link l_forearm_mtb_acc_1b9
- added link r_forearm_mtb_acc_2b7
- added link r_forearm_mtb_acc_2b8
- added link r_forearm_mtb_acc_2b9
Joints:
- removed joint SIM_SEA_2-5_L_ELBOW--SIM_SEA_2-5_L_ELBOW_PROSUP
- added joint l_elbow: type revolute, parent l_upper_arm, child l_elbow_1, origin xyz=0 0.0339999 0.07926 rpy=0 -1.30899700697 -3.14159265359, axis 2.22044604925e-16 -1.0 0.0, limit lower=0.261799387799 upper=1.85004900711 effort=50000 velocity=50000
- added joint l_forearm_mtb_acc_1b7_fixed_joint: type fixed, parent l_forearm, child l_forearm_mtb_acc_1b7, origin xyz=0.0759068847722 -0.005483 -0.0113068281789 rpy=0.26179949998 0.000370413042328 -1.57033448496
- added joint l_forearm_mtb_acc_1b8_fixed_joint: type fixed, parent l_forearm, child l_forearm_mtb_acc_1b8, origin xyz=0.0504582616754 -0.0180279 0.040491856636 rpy=-0.661143946092 0.147825248461 -3.04952253889
- added joint l_forearm_mtb_acc_1b9_fixed_joint: type fixed, parent l_forearm, child l_forearm_mtb_acc_1b9, origin xyz=0.0211332875376 0.025657 -0.0153763398932 rpy=1.76682134218 0.261099829847 3.08752548202
- added joint r_forearm_mtb_acc_2b7_fixed_joint: type fixed, parent r_forearm, child r_forearm_mtb_acc_2b7, origin xyz=-0.0759068847722 0.005497 -0.0113068281789 rpy=0.26179949998 0.000370413042328 1.57125816863
- added joint r_forearm_mtb_acc_2b8_fixed_joint: type fixed, parent r_forearm, child r_forearm_mtb_acc_2b8, origin xyz=-0.0507255655432 -0.0187484 0.040023592236 rpy=0.661159832193 0.147746087249 -0.0919671195152
- added joint r_forearm_mtb_acc_2b9_fixed_joint: type fixed, parent r_forearm, child r_forearm_mtb_acc_2b9, origin xyz=-0.0206720957139 0.027924 -0.0135079409739 rpy=-1.76682626732 0.261191225646 0.054048344372

File: generated/robots/iCubGenova02/model.urdf (robot description, URDF)
Before this commit: robot ICUB_2-5_BB_SIM_MODEL, 107 links, 106 joints
Links:
- added link l_forearm_mtb_acc_1b7
- added link l_forearm_mtb_acc_1b8
- added link l_forearm_mtb_acc_1b9
- added link r_forearm_mtb_acc_2b7
- added link r_forearm_mtb_acc_2b8
- added link r_forearm_mtb_acc_2b9
Joints:
- removed joint SIM_SEA_2-5_L_ELBOW--SIM_SEA_2-5_L_ELBOW_PROSUP
- added joint l_elbow: type revolute, parent l_upper_arm, child l_elbow_1, origin xyz=0 0.0339999 0.07926 rpy=0 -1.30899700697 -3.14159265359, axis 2.22044604925e-16 -1.0 0.0, limit lower=0.261799387799 upper=1.85004900711 effort=50000 velocity=50000
- added joint l_forearm_mtb_acc_1b7_fixed_joint: type fixed, parent l_forearm, child l_forearm_mtb_acc_1b7, origin xyz=0.0759068847722 -0.005483 -0.0113068281789 rpy=0.26179949998 0.000370413042328 -1.57033448496
- added joint l_forearm_mtb_acc_1b8_fixed_joint: type fixed, parent l_forearm, child l_forearm_mtb_acc_1b8, origin xyz=0.0504582616754 -0.0180279 0.040491856636 rpy=-0.661143946092 0.147825248461 -3.04952253889
- added joint l_forearm_mtb_acc_1b9_fixed_joint: type fixed, parent l_forearm, child l_forearm_mtb_acc_1b9, origin xyz=0.0211332875376 0.025657 -0.0153763398932 rpy=1.76682134218 0.261099829847 3.08752548202
- added joint r_forearm_mtb_acc_2b7_fixed_joint: type fixed, parent r_forearm, child r_forearm_mtb_acc_2b7, origin xyz=-0.0759068847722 0.005497 -0.0113068281789 rpy=0.26179949998 0.000370413042328 1.57125816863
- added joint r_forearm_mtb_acc_2b8_fixed_joint: type fixed, parent r_forearm, child r_forearm_mtb_acc_2b8, origin xyz=-0.0507255655432 -0.0187484 0.040023592236 rpy=0.661159832193 0.147746087249 -0.0919671195152
- added joint r_forearm_mtb_acc_2b9_fixed_joint: type fixed, parent r_forearm, child r_forearm_mtb_acc_2b9, origin xyz=-0.0206720957139 0.027924 -0.0135079409739 rpy=-1.76682626732 0.261191225646 0.054048344372
