Commit message: adding forearm dh frames and updating all models

File: generated/robots/iCubDarmstadt01/model.urdf (robot description, URDF)
Before this commit: robot ICUB_2-5_BB_SIM_MODEL, 113 links, 112 joints
Links:
- added link l_forearm_dh_frame
- added link l_forearm_skin_0
- added link l_forearm_skin_1
- added link l_forearm_skin_10
- added link l_forearm_skin_11
- added link l_forearm_skin_12
- added link l_forearm_skin_13
- added link l_forearm_skin_14
- added link l_forearm_skin_15
- added link l_forearm_skin_16
- added link l_forearm_skin_17
- added link l_forearm_skin_19
- added link l_forearm_skin_2
- added link l_forearm_skin_22
- added link l_forearm_skin_24
- added link l_forearm_skin_25
- added link l_forearm_skin_28
- added link l_forearm_skin_29
- added link l_forearm_skin_3
- added link l_forearm_skin_4
- added link l_forearm_skin_5
- added link l_forearm_skin_6
- added link l_forearm_skin_7
- added link l_forearm_skin_8
- added link l_forearm_skin_9
- added link r_forearm_dh_frame
- added link r_forearm_skin_0
- added link r_forearm_skin_1
- added link r_forearm_skin_10
- added link r_forearm_skin_11
- added link r_forearm_skin_12
- added link r_forearm_skin_13
- added link r_forearm_skin_14
- added link r_forearm_skin_15
- added link r_forearm_skin_16
- added link r_forearm_skin_17
- added link r_forearm_skin_19
- added link r_forearm_skin_2
- added link r_forearm_skin_22
- added link r_forearm_skin_24
- added link r_forearm_skin_25
- added link r_forearm_skin_28
- added link r_forearm_skin_29
- added link r_forearm_skin_3
- added link r_forearm_skin_4
- added link r_forearm_skin_5
- added link r_forearm_skin_6
- added link r_forearm_skin_7
- added link r_forearm_skin_8
- added link r_forearm_skin_9
- link l_forearm: mass 0.635334 -> 0.636185
- link r_forearm: mass 0.63385 -> 0.6347
Joints:
- added joint l_forearm_dh_frame_fixed_joint: type fixed, parent l_forearm, child l_forearm_dh_frame, origin xyz=0.102871102373 7.00000000002e-06 0.0275642213111 rpy=2.87979333376 0 1.57079632679
- added joint l_forearm_skin_0_fixed_joint: type fixed, parent l_forearm, child l_forearm_skin_0, origin xyz=0.0454493286618 -0.0323169 -0.00628656037901 rpy=1.69181522292 -0.271026744341 0.0727882713185
- added joint l_forearm_skin_10_fixed_joint: type fixed, parent l_forearm, child l_forearm_skin_10, origin xyz=0.0542285469707 0.007546 -0.0321470048792 rpy=-2.94123313406 -0.328304471922 -0.0139662781936
- added joint l_forearm_skin_11_fixed_joint: type fixed, parent l_forearm, child l_forearm_skin_11, origin xyz=0.0542241170843 -0.0112832 -0.0321432225378 rpy=2.93929835957 -0.329101389745 0.0142734891292
- added joint l_forearm_skin_12_fixed_joint: type fixed, parent l_forearm, child l_forearm_skin_12, origin xyz=0.0375994892687 -0.0204556 -0.0340192145887 rpy=2.58303505964 -0.29483050207 0.021326850448
- added joint l_forearm_skin_13_fixed_joint: type fixed, parent l_forearm, child l_forearm_skin_13, origin xyz=0.0228551127224 -0.0112878 -0.0418919975134 rpy=2.94896679198 -0.270583947189 0.00177385006765
- added joint l_forearm_skin_14_fixed_joint: type fixed, parent l_forearm, child l_forearm_skin_14, origin xyz=0.0687703535183 -0.0193999 -0.0230240524437 rpy=2.52462250363 -0.387794511771 0.0912924111683
- added joint l_forearm_skin_15_fixed_joint: type fixed, parent l_forearm, child l_forearm_skin_15, origin xyz=0.0633786419662 -0.0293843 -0.00879405455544 rpy=1.80492769741 -0.289783281916 0.113933739306
- added joint l_forearm_skin_16_fixed_joint: type fixed, parent l_forearm, child l_forearm_skin_16, origin xyz=0.03792482187 -0.0327268 0.0206369503605 rpy=1.41280007026 -0.25082462139 0.0758652301584
- added joint l_forearm_skin_17_fixed_joint: type fixed, parent l_forearm, child l_forearm_skin_17, origin xyz=0.0543170548821 -0.0299646 0.0303291240179 rpy=1.27223716205 -0.23059304703 0.109637225219
- added joint l_forearm_skin_19_fixed_joint: type fixed, parent l_forearm, child l_forearm_skin_19, origin xyz=0.0381266365957 0.029054 0.0206905088005 rpy=-1.41560888703 -0.252569290226 -0.0644404747027
- added joint l_forearm_skin_1_fixed_joint: type fixed, parent l_forearm, child l_forearm_skin_1, origin xyz=0.0333729194645 -0.0310662 -0.0198457833637 rpy=1.86694023278 -0.274442533764 0.0421228737473
- added joint l_forearm_skin_22_fixed_joint: type fixed, parent l_forearm, child l_forearm_skin_22, origin xyz=0.054417420924 0.026483 0.0306036550683 rpy=-1.2658242728 -0.234328151379 -0.0937094738802
- added joint l_forearm_skin_24_fixed_joint: type fixed, parent l_forearm, child l_forearm_skin_24, origin xyz=0.0700345474855 0.007477 0.0500690507585 rpy=-0.23489327644 -0.0388172993982 -0.0548291989999
- added joint l_forearm_skin_25_fixed_joint: type fixed, parent l_forearm, child l_forearm_skin_25, origin xyz=0.0535999345704 0.015984 0.0454697642082 rpy=-0.564295527715 -0.136980272197 -0.0819608256656
- added joint l_forearm_skin_28_fixed_joint: type fixed, parent l_forearm, child l_forearm_skin_28, origin xyz=0.0535859427439 -0.0196522 0.0453519794414 rpy=0.579311106949 -0.133994306778 0.0867597858312
- added joint l_forearm_skin_29_fixed_joint: type fixed, parent l_forearm, child l_forearm_skin_29, origin xyz=0.0700355934441 -0.0111936 0.050011055327 rpy=0.248630982209 -0.0383136556786 0.0583026624266
- added joint l_forearm_skin_2_fixed_joint: type fixed, parent l_forearm, child l_forearm_skin_2, origin xyz=0.0146989188671 -0.0335184 -0.0160118304296 rpy=1.72847287019 -0.264015219116 0.0142600467197
- added joint l_forearm_skin_3_fixed_joint: type fixed, parent l_forearm, child l_forearm_skin_3, origin xyz=0.0455673195039 0.028651 -0.00633010588609 rpy=-1.69487280859 -0.269757727104 -0.061995217851
- added joint l_forearm_skin_4_fixed_joint: type fixed, parent l_forearm, child l_forearm_skin_4, origin xyz=0.0635326591815 0.025877 -0.00899793917324 rpy=-1.81747870108 -0.287406884885 -0.0998316152826
- added joint l_forearm_skin_5_fixed_joint: type fixed, parent l_forearm, child l_forearm_skin_5, origin xyz=0.0688211941968 0.015709 -0.0231133361791 rpy=-2.5410475806 -0.385627260642 -0.0867227569203
- added joint l_forearm_skin_6_fixed_joint: type fixed, parent l_forearm, child l_forearm_skin_6, origin xyz=0.0333948695074 0.027308 -0.0198326549359 rpy=-1.86628164653 -0.272886336181 -0.0371068033783
- added joint l_forearm_skin_7_fixed_joint: type fixed, parent l_forearm, child l_forearm_skin_7, origin xyz=0.0147224518893 0.029702 -0.0159327448629 rpy=-1.72564640857 -0.263992900722 -0.0143801109253
- added joint l_forearm_skin_8_fixed_joint: type fixed, parent l_forearm, child l_forearm_skin_8, origin xyz=0.0228528628554 0.007546 -0.041885146375 rpy=-2.94801979137 -0.270605090512 -0.00178708074348
- added joint l_forearm_skin_9_fixed_joint: type fixed, parent l_forearm, child l_forearm_skin_9, origin xyz=0.0376032734683 0.016715 -0.0340163371186 rpy=-2.58406517708 -0.2933217196 -0.0203085796276
- added joint r_forearm_dh_frame_fixed_joint: type fixed, parent r_forearm, child r_forearm_dh_frame, origin xyz=-0.102871102373 7.00000000002e-06 0.0275642213111 rpy=-0.261799319827 0 -1.57079632679
- added joint r_forearm_skin_0_fixed_joint: type fixed, parent r_forearm, child r_forearm_skin_0, origin xyz=-0.0454493286618 0.030077 -0.00628656037901 rpy=1.69181522292 -0.271026744341 -3.06880438227
- added joint r_forearm_skin_10_fixed_joint: type fixed, parent r_forearm, child r_forearm_skin_10, origin xyz=-0.0542285469707 -0.0097861 -0.0321470048792 rpy=-2.94123313406 -0.328304471922 3.1276263754
- added joint r_forearm_skin_11_fixed_joint: type fixed, parent r_forearm, child r_forearm_skin_11, origin xyz=-0.0542241170843 0.009043 -0.0321432225378 rpy=2.93929835957 -0.329101389745 -3.12731916446
- added joint r_forearm_skin_12_fixed_joint: type fixed, parent r_forearm, child r_forearm_skin_12, origin xyz=-0.0375994892687 0.018216 -0.0340192145887 rpy=2.58303505964 -0.29483050207 -3.12026580314
- added joint r_forearm_skin_13_fixed_joint: type fixed, parent r_forearm, child r_forearm_skin_13, origin xyz=-0.0228551127224 0.009048 -0.0418919975134 rpy=2.94896679198 -0.270583947189 -3.13981880352
- added joint r_forearm_skin_14_fixed_joint: type fixed, parent r_forearm, child r_forearm_skin_14, origin xyz=-0.0687703535183 0.01716 -0.0230240524437 rpy=2.48044991868 -0.295542566281 -2.91877349139
- added joint r_forearm_skin_15_fixed_joint: type fixed, parent r_forearm, child r_forearm_skin_15, origin xyz=-0.0633786419662 0.027145 -0.00879405455544 rpy=1.80492769741 -0.289783281916 -3.02765891428
- added joint r_forearm_skin_16_fixed_joint: type fixed, parent r_forearm, child r_forearm_skin_16, origin xyz=-0.03792482187 0.030487 0.0206369503605 rpy=1.41280007026 -0.25082462139 -3.06572742343
- added joint r_forearm_skin_17_fixed_joint: type fixed, parent r_forearm, child r_forearm_skin_17, origin xyz=-0.0543170548821 0.027725 0.0303291240179 rpy=1.27223716205 -0.23059304703 -3.03195542837
- added joint r_forearm_skin_19_fixed_joint: type fixed, parent r_forearm, child r_forearm_skin_19, origin xyz=-0.0381266365957 -0.0312941 0.0206905088005 rpy=-1.41560888703 -0.252569290226 3.07715217889
- added joint r_forearm_skin_1_fixed_joint: type fixed, parent r_forearm, child r_forearm_skin_1, origin xyz=-0.0333729194645 0.028826 -0.0198457833637 rpy=1.86694023278 -0.274442533764 -3.09946977984
- added joint r_forearm_skin_22_fixed_joint: type fixed, parent r_forearm, child r_forearm_skin_22, origin xyz=-0.054417420924 -0.0287223 0.0306036550683 rpy=-1.2658242728 -0.234328151379 3.04788317971
- added joint r_forearm_skin_24_fixed_joint: type fixed, parent r_forearm, child r_forearm_skin_24, origin xyz=-0.0700345474855 -0.0097164 0.0500690507585 rpy=-0.23489327644 -0.0388172993982 3.08676345459
- added joint r_forearm_skin_25_fixed_joint: type fixed, parent r_forearm, child r_forearm_skin_25, origin xyz=-0.0535999345704 -0.0182238 0.0454697642082 rpy=-0.564295527715 -0.136980272197 3.05963182792
- added joint r_forearm_skin_28_fixed_joint: type fixed, parent r_forearm, child r_forearm_skin_28, origin xyz=-0.0535859427439 0.017412 0.0453519794414 rpy=0.59077064408 -0.0531607226063 3.10597081167
- added joint r_forearm_skin_29_fixed_joint: type fixed, parent r_forearm, child r_forearm_skin_29, origin xyz=-0.0700355934441 0.008954 0.050011055327 rpy=0.248630982209 -0.0383136556786 -3.08328999116
- added joint r_forearm_skin_2_fixed_joint: type fixed, parent r_forearm, child r_forearm_skin_2, origin xyz=-0.0146989188671 0.031279 -0.0160118304296 rpy=1.72847287019 -0.264015219116 -3.12733260687
- added joint r_forearm_skin_3_fixed_joint: type fixed, parent r_forearm, child r_forearm_skin_3, origin xyz=-0.0455673195039 -0.030891 -0.00633010588609 rpy=-1.69487280859 -0.269757727104 3.07959743574
- added joint r_forearm_skin_4_fixed_joint: type fixed, parent r_forearm, child r_forearm_skin_4, origin xyz=-0.0635326591815 -0.0281163 -0.00899793917324 rpy=-1.80734960194 -0.0393131796327 2.97997643632
- added joint r_forearm_skin_5_fixed_joint: type fixed, parent r_forearm, child r_forearm_skin_5, origin xyz=-0.0688211941968 -0.0179483 -0.0231133361791 rpy=-2.5410475806 -0.385627260642 3.05486989667
- added joint r_forearm_skin_6_fixed_joint: type fixed, parent r_forearm, child r_forearm_skin_6, origin xyz=-0.0333948695074 -0.0295479 -0.0198326549359 rpy=-1.86628164653 -0.272886336181 3.10448585021
- added joint r_forearm_skin_7_fixed_joint: type fixed, parent r_forearm, child r_forearm_skin_7, origin xyz=-0.0147224518893 -0.0319422 -0.0159327448629 rpy=-1.72564640857 -0.263992900722 3.12721254266
- added joint r_forearm_skin_8_fixed_joint: type fixed, parent r_forearm, child r_forearm_skin_8, origin xyz=-0.0228528628554 -0.0097862 -0.041885146375 rpy=-2.94801979137 -0.270605090512 3.13980557285
- added joint r_forearm_skin_9_fixed_joint: type fixed, parent r_forearm, child r_forearm_skin_9, origin xyz=-0.0376032734683 -0.018955 -0.0340163371186 rpy=-2.58406517708 -0.2933217196 3.12128407396
- joint l_ankle_pitch: origin xyz=0.0592832 -0.201 0 rpy=0 0 0 -> xyz=0.0406034 -0.2005 0 rpy=0 0 0
- joint l_ankle_roll: origin xyz=-0.0355 0 0.04808755 rpy=0 0 0 -> xyz=-0.0270179 0 0.04808755 rpy=0 0 0
- joint l_forearm_mtb_acc_1b7_fixed_joint: origin xyz=0.0759068847722 -0.005483 -0.0113068281789 rpy=0.26179949998 0.000370413042328 -1.57033448496 -> xyz=0.0768728106161 -0.005483 -0.0110480091994 rpy=0.26179949998 0.000370413042328 -1.57033448496
- joint l_forearm_mtb_acc_1b8_fixed_joint: origin xyz=0.0504582616754 -0.0180279 0.040491856636 rpy=-0.661143946092 0.147825248461 -3.04952253889 -> xyz=0.0514241875192 -0.0180279 0.0407506756155 rpy=-0.661143946092 0.147825248461 -3.04952253889
- joint l_forearm_mtb_acc_1b9_fixed_joint: origin xyz=0.0211332875376 0.025657 -0.0153763398932 rpy=1.76682134218 0.261099829847 3.08752548202 -> xyz=0.0220992133815 0.025657 -0.0151175209138 rpy=1.76682134218 0.261099829847 3.08752548202
- joint l_knee: axis -1.0 -0.0 -0.0 -> -1.0 0.0 0.0; origin xyz=-0.0237832 -0.145625 0 rpy=0 0 0 -> xyz=-0.0135855 -0.145625 0 rpy=0 0 0
- joint l_lower_leg_ems_acc_eb7_fixed_joint: origin xyz=0.0350978 -0.092765 0.04351373 rpy=0 -0.218166543341 1.57079632679 -> xyz=0.0249001 -0.092765 0.04351373 rpy=0 -0.218166543341 1.57079632679
- joint l_lower_leg_ems_gyro_eb7_fixed_joint: origin xyz=0.0356017 -0.088301 0.044503292 rpy=0 -0.218166543341 1.57079632679 -> xyz=0.025404 -0.088301 0.044503292 rpy=0 -0.218166543341 1.57079632679
- joint l_lower_leg_mtb_acc_10b10_fixed_joint: origin xyz=0.030989 -0.011037 0.05238133 rpy=-1.32645042367 0 1.57079632679 -> xyz=0.0563295 -0.043468 0.0259151 rpy=1.30899714594 -0.000112159802878 1.57082638021
- joint l_lower_leg_mtb_acc_10b11_fixed_joint: origin xyz=-0.0179355 -0.092958 0.0184593 rpy=-1.3089971472 -2.54317885716e-05 1.57078951235 -> xyz=-0.0281332 -0.092958 0.0184593 rpy=-1.3089971472 -2.54317885716e-05 1.57078951235
- joint l_lower_leg_mtb_acc_10b8_fixed_joint: origin xyz=0.0099841 -0.004318 0.0544518 rpy=-0.349065638045 3.97141037841e-05 1.57090544048 -> xyz=0.0307696 -0.004318 0.05313347 rpy=0.24434616607 0 1.57079632679
- joint l_lower_leg_mtb_acc_10b9_fixed_joint: origin xyz=0.0665272 -0.043468 0.0259151 rpy=1.30899714594 -0.000112159802878 1.57082638021 -> xyz=-0.0002136 -0.004318 0.0544518 rpy=-0.349065638045 3.97141037841e-05 1.57090544048
- joint l_upper_leg_mtb_acc_10b2_fixed_joint: origin xyz=0.0083839 0.039452 0.05335544 rpy=0.837758036965 -8.62912869137e-05 1.57087402394 -> xyz=0.0083839 0.039452 0.05335544 rpy=0.261799318135 -3.00531353284e-05 1.57090848663
- joint l_wrist_pitch: origin xyz=0.0938586368089 7.00000000002e-06 0.0573355055587 rpy=0 0 0 -> xyz=0.103427563179 7.00000000002e-06 0.0254874807467 rpy=0 0 0
- joint l_wrist_yaw: origin xyz=0.00796889402672 -0.0194999 -0.0297403254739 rpy=0 0 0 -> xyz=-0.000634106499644 -0.0194999 0.00236651831751 rpy=0 0 0
- joint r_ankle_pitch: origin xyz=-0.0593039 -0.201 0 rpy=0 0 0 -> xyz=-0.0188325 -0.2005 0 rpy=0 0 0
- joint r_ankle_roll: axis -0.0 -0.0 -1.0 -> 0.0 0.0 -1.0; origin xyz=0.0355 0 -0.0185 rpy=0 0 0 -> xyz=0.0285 0 -0.0185 rpy=0 0 0
- joint r_forearm_mtb_acc_2b7_fixed_joint: origin xyz=-0.0759068847722 0.005497 -0.0113068281789 rpy=0.26179949998 0.000370413042328 1.57125816863 -> xyz=-0.0768728106161 0.005497 -0.0110480091994 rpy=0.26179949998 0.000370413042328 1.57125816863
- joint r_forearm_mtb_acc_2b8_fixed_joint: origin xyz=-0.0507255655432 -0.0187484 0.040023592236 rpy=0.661159832193 0.147746087249 -0.0919671195152 -> xyz=-0.0514186285381 0.015786 0.0407521034996 rpy=-0.661143946092 0.147825248461 0.092070114703
- joint r_forearm_mtb_acc_2b9_fixed_joint: origin xyz=-0.0206720957139 0.027924 -0.0135079409739 rpy=-1.76682626732 0.261191225646 0.054048344372 -> xyz=-0.0216380215578 0.027924 -0.0132491219944 rpy=-1.76682626732 0.261191225646 0.054048344372
- joint r_hip_pitch: axis -1.0 -0.0 -0.0 -> -1.0 0.0 0.0
- joint r_hip_roll: axis -0.0 -0.0 -1.0 -> 0.0 0.0 -1.0
- joint r_knee: origin xyz=0.0238039 -0.145625 0 rpy=0 0 0 -> xyz=-0.0096675 -0.145625 0 rpy=0 0 0
- joint r_lower_leg_ems_acc_eb9_fixed_joint: origin xyz=-0.0099643 -0.092765 0.04351373 rpy=0 -0.218166543341 1.57079632679 -> xyz=0.0235071 -0.092765 0.04351373 rpy=0 -0.218166543341 1.57079632679
- joint r_lower_leg_ems_gyro_eb9_fixed_joint: origin xyz=-0.0094604 -0.088301 0.044503292 rpy=0 -0.218166543341 1.57079632679 -> xyz=0.024011 -0.088301 0.044503292 rpy=0 -0.218166543341 1.57079632679
- joint r_lower_leg_mtb_acc_11b10_fixed_joint: origin xyz=-0.0389997 -0.004318 0.05362922 rpy=-0.244346164565 2.80911040962e-05 1.57090899435 -> xyz=-0.0325465 -0.043468 0.0278945 rpy=-1.30899714732 0 1.57079632679
- joint r_lower_leg_mtb_acc_11b11_fixed_joint: origin xyz=0.0184451 -0.092958 0.0164801 rpy=1.30899714594 -0.000112159802878 1.57082638021 -> xyz=0.0519165 -0.092958 0.0164801 rpy=1.30899714594 -0.000112159802878 1.57082638021
- joint r_lower_leg_mtb_acc_11b8_fixed_joint: origin xyz=-0.008081 -0.004318 0.0537517 rpy=0.349065638046 -3.97141043948e-05 1.57090544048 -> xyz=-0.0055283 -0.004318 0.05362922 rpy=-0.244346164565 2.80911040962e-05 1.57090899435
- joint r_lower_leg_mtb_acc_11b9_fixed_joint: origin xyz=-0.0660179 -0.043468 0.0278945 rpy=-1.30899714732 0 1.57079632679 -> xyz=0.0253904 -0.004318 0.0537517 rpy=0.349065638045 -3.97141037841e-05 1.57090544048
- joint r_upper_leg_mtb_acc_11b2_fixed_joint: origin xyz=-0.0064065 0.039256 0.0539467 rpy=-0.837758053858 -0.000342790749344 1.57087401652 -> xyz=-0.0064065 0.039256 0.0539467 rpy=-0.261799341927 -0.000399050135154 1.57090848318
- joint r_wrist_pitch: origin xyz=-0.102539283029 7.00000000002e-06 0.0249388840141 rpy=0 0 0 -> xyz=-0.103505208873 7.00000000002e-06 0.0251977029936 rpy=0 0 0

File: generated/robots/iCubGenova02/model.urdf (robot description, URDF)
Before this commit: robot ICUB_2-5_BB_SIM_MODEL, 161 links, 160 joints
Links:
- added link l_forearm_dh_frame
- added link r_forearm_dh_frame
Joints:
- added joint l_forearm_dh_frame_fixed_joint: type fixed, parent l_forearm, child l_forearm_dh_frame, origin xyz=0.102871102373 7.00000000002e-06 0.0275642213111 rpy=2.87979333376 0 1.57079632679
- added joint r_forearm_dh_frame_fixed_joint: type fixed, parent r_forearm, child r_forearm_dh_frame, origin xyz=-0.102871102373 7.00000000002e-06 0.0275642213111 rpy=-0.261799319827 0 -1.57079632679
