Commit message: fixing definition of missing meshes (l/r_upper_thigh and lap_belt_2)

File: generated/robots/iCubDarmstadt01/model.urdf (robot description, URDF)
Before this commit: robot ICUB_2-5_BB_SIM_MODEL, 163 links, 162 joints
Links:
- link l_hip_3: geometry collision mesh filename=model://iCubGenova02/meshes/dae/sim_sea_2-5_l_upper_thigh_p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 scale=0.001 0.001 0.001; visual mesh filename=model://iCubGenova02/meshes/dae/sim_sea_2-5_l_upper_thigh_p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 scale=0.001 0.001 0.001
- link r_hip_3: geometry collision mesh filename=model://iCubGenova02/meshes/dae/sim_sea_2-5_r_upper_thigh_p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 scale=0.001 0.001 0.001; visual mesh filename=model://iCubGenova02/meshes/dae/sim_sea_2-5_r_upper_thigh_p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 scale=0.001 0.001 0.001
- link torso_2: mass 0.428161 -> 0.425685; geometry collision mesh filename=model://iCubGenova02/meshes/dae/sim_sea_2-5_lap_belt_2_prt.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 scale=0.001 0.001 0.001; visual mesh filename=model://iCubGenova02/meshes/dae/sim_sea_2-5_lap_belt_2_prt.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 scale=0.001 0.001 0.001
Joints:
- joint chest_ems_acc_eb1_fixed_joint: origin xyz=0.0647855001907 0.064043 -0.064709 rpy=3.1415169123 -0.261799309122 0.000292641880255 -> xyz=0.0647855001907 0.064043 -0.0647091 rpy=3.1415169123 -0.261799309122 0.000292641880255
- joint chest_ems_acc_eb4_fixed_joint: origin xyz=-0.0621620998093 0.088063 -0.0529886 rpy=-3.14159050476 -0.261799319819 3.14158433987 -> xyz=-0.0621620998093 0.088063 -0.0529887 rpy=-3.14159050476 -0.261799319819 3.14158433987
- joint chest_ems_gyro_eb1_fixed_joint: origin xyz=0.0692016001907 0.064548 -0.0635257 rpy=3.1415169123 -0.261799309122 0.000292641880255 -> xyz=0.0692016001907 0.064548 -0.0635258 rpy=3.1415169123 -0.261799309122 0.000292641880255
- joint chest_ems_gyro_eb2_fixed_joint: origin xyz=0.0160371001907 0.087559 -0.0653478 rpy=3.14159050104 0.261799319819 3.14158433678 -> xyz=0.0160371001907 0.087559 -0.0653479 rpy=3.14159050104 0.261799319819 3.14158433678
- joint chest_ems_gyro_eb4_fixed_joint: origin xyz=-0.0665783998093 0.087559 -0.0518053 rpy=-3.14159050476 -0.261799319819 3.14158433987 -> xyz=-0.0665783998093 0.087559 -0.0518054 rpy=-3.14159050476 -0.261799319819 3.14158433987
- joint chest_mtb_acc_0b10_fixed_joint: origin xyz=0.0594286001907 -0.0018543 0.0457982 rpy=-0.875168153475 0.116362025479 -1.65561807505 -> xyz=0.0594286001907 -0.0018543 0.0457981 rpy=-0.875168153475 0.116362025479 -1.65561807505
- joint chest_mtb_acc_0b7_fixed_joint: origin xyz=-0.0607539998093 -0.0017836 0.0442342 rpy=0.875167771492 0.116363734392 -1.48597350247 -> xyz=-0.0607539998093 -0.0017836 0.0442341 rpy=0.875167771492 0.116363734392 -1.48597350247
- joint l_forearm_mtb_acc_1b7_fixed_joint: origin xyz=0.0768728106161 -0.005483 -0.0110480091994 rpy=0.26179949998 0.000370413042328 -1.57033448496 -> xyz=0.0768727847342 -0.005483 -0.0110479126068 rpy=0.26179949998 0.000370413042328 -1.57033448496
- joint l_forearm_mtb_acc_1b8_fixed_joint: origin xyz=0.0514241875192 -0.0180279 0.0407506756155 rpy=-0.661143946092 0.147825248461 -3.04952253889 -> xyz=0.0514241740607 -0.0180279 0.0407507258436 rpy=-0.661143946092 0.147825248461 -3.04952253889
- joint l_forearm_mtb_acc_1b9_fixed_joint: origin xyz=0.0220992133815 0.025657 -0.0151175209138 rpy=1.76682134218 0.261099829847 3.08752548202 -> xyz=0.0220991874996 0.025657 -0.0151174243212 rpy=1.76682134218 0.261099829847 3.08752548202
- joint l_forearm_skin_10_fixed_joint: origin xyz=0.0542285469707 0.007546 -0.0321470048792 rpy=-2.94123313406 -0.328304471922 -0.0139662781936 -> xyz=0.0542285210888 0.007546 -0.0321469082866 rpy=-2.94123313406 -0.328304471922 -0.0139662781936
- joint l_forearm_skin_11_fixed_joint: origin xyz=0.0542241170843 -0.0112832 -0.0321432225378 rpy=2.93929835957 -0.329101389745 0.0142734891292 -> xyz=0.0542240912024 -0.0112832 -0.0321431259452 rpy=2.93929835957 -0.329101389745 0.0142734891292
- joint l_forearm_skin_12_fixed_joint: origin xyz=0.0375994892687 -0.0204556 -0.0340192145887 rpy=2.58303505964 -0.29483050207 0.021326850448 -> xyz=0.0375994633868 -0.0204556 -0.0340191179961 rpy=2.58303505964 -0.29483050207 0.021326850448
- joint l_forearm_skin_13_fixed_joint: origin xyz=0.0228551127224 -0.0112878 -0.0418919975134 rpy=2.94896679198 -0.270583947189 0.00177385006765 -> xyz=0.0228550868405 -0.0112878 -0.0418919009209 rpy=2.94896679198 -0.270583947189 0.00177385006765
- joint l_forearm_skin_14_fixed_joint: origin xyz=0.0687703535183 -0.0193999 -0.0230240524437 rpy=2.52462250363 -0.387794511771 0.0912924111683 -> xyz=0.0687703276364 -0.0193999 -0.0230239558511 rpy=2.52462250363 -0.387794511771 0.0912924111683
- joint l_forearm_skin_19_fixed_joint: origin xyz=0.0381266365957 0.029054 0.0206905088005 rpy=-1.41560888703 -0.252569290226 -0.0644404747027 -> xyz=0.0381266107138 0.029054 0.020690605393 rpy=-1.41560888703 -0.252569290226 -0.0644404747027
- joint l_forearm_skin_1_fixed_joint: origin xyz=0.0333729194645 -0.0310662 -0.0198457833637 rpy=1.86694023278 -0.274442533764 0.0421228737473 -> xyz=0.0333728935826 -0.0310662 -0.0198456867711 rpy=1.86694023278 -0.274442533764 0.0421228737473
- joint l_forearm_skin_22_fixed_joint: origin xyz=0.054417420924 0.026483 0.0306036550683 rpy=-1.2658242728 -0.234328151379 -0.0937094738802 -> xyz=0.0544173950421 0.026483 0.0306037516609 rpy=-1.2658242728 -0.234328151379 -0.0937094738802
- joint l_forearm_skin_24_fixed_joint: origin xyz=0.0700345474855 0.007477 0.0500690507585 rpy=-0.23489327644 -0.0388172993982 -0.0548291989999 -> xyz=0.0700345319564 0.007477 0.050069108714 rpy=-0.23489327644 -0.0388172993982 -0.0548291989999
- joint l_forearm_skin_25_fixed_joint: origin xyz=0.0535999345704 0.015984 0.0454697642082 rpy=-0.564295527715 -0.136980272197 -0.0819608256656 -> xyz=0.0535999216295 0.015984 0.0454698125045 rpy=-0.564295527715 -0.136980272197 -0.0819608256656
- joint l_forearm_skin_28_fixed_joint: origin xyz=0.0535859427439 -0.0196522 0.0453519794414 rpy=0.579311106949 -0.133994306778 0.0867597858312 -> xyz=0.0535859272148 -0.0196522 0.045352037397 rpy=0.579311106949 -0.133994306778 0.0867597858312
- joint l_forearm_skin_29_fixed_joint: origin xyz=0.0700355934441 -0.0111936 0.050011055327 rpy=0.248630982209 -0.0383136556786 0.0583026624266 -> xyz=0.0700355805031 -0.0111936 0.0500111036233 rpy=0.248630982209 -0.0383136556786 0.0583026624266
- joint l_forearm_skin_2_fixed_joint: origin xyz=0.0146989188671 -0.0335184 -0.0160118304296 rpy=1.72847287019 -0.264015219116 0.0142600467197 -> xyz=0.0146988929852 -0.0335184 -0.0160117338371 rpy=1.72847287019 -0.264015219116 0.0142600467197
- joint l_forearm_skin_3_fixed_joint: origin xyz=0.0455673195039 0.028651 -0.00633010588609 rpy=-1.69487280859 -0.269757727104 -0.061995217851 -> xyz=0.045567293622 0.028651 -0.00633000929351 rpy=-1.69487280859 -0.269757727104 -0.061995217851
- joint l_forearm_skin_4_fixed_joint: origin xyz=0.0635326591815 0.025877 -0.00899793917324 rpy=-1.81747870108 -0.287406884885 -0.0998316152826 -> xyz=0.0635326332996 0.025877 -0.00899784258066 rpy=-1.81747870108 -0.287406884885 -0.0998316152826
- joint l_forearm_skin_6_fixed_joint: origin xyz=0.0333948695074 0.027308 -0.0198326549359 rpy=-1.86628164653 -0.272886336181 -0.0371068033783 -> xyz=0.0333948436255 0.027308 -0.0198325583433 rpy=-1.86628164653 -0.272886336181 -0.0371068033783
- joint l_forearm_skin_7_fixed_joint: origin xyz=0.0147224518893 0.029702 -0.0159327448629 rpy=-1.72564640857 -0.263992900722 -0.0143801109253 -> xyz=0.0147224260074 0.029702 -0.0159326482703 rpy=-1.72564640857 -0.263992900722 -0.0143801109253
- joint l_hand_dh_frame_fixed_joint: origin xyz=0.0576543237247 -0.0055568 0.0136937357157 rpy=-1.57079632679 -0.261799319827 0 -> xyz=0.0576542978428 -0.0055568 0.0136938323083 rpy=-1.57079632679 -0.261799319827 0
- joint l_shoulder_pitch: origin xyz=0.120016000191 0.0928 0.0079694 rpy=0 0 0 -> xyz=0.120016000191 0.0928 0.0079693 rpy=0 0 0
- joint l_shoulder_roll: origin xyz=-0.013671 0 0.0085203 rpy=0.270597317916 0.252680177542 -1.50155688559 -> xyz=-0.013671 0 0.0085204 rpy=0.270597317916 0.252680177542 -1.50155688559
- joint l_shoulder_yaw: origin xyz=0.0253143218312 1.37518334151e-07 -0.00540052326137 rpy=-0.252689546175 -0.0085186183214 -0.067039889142 -> xyz=0.0253143468312 1.11636438205e-07 -0.00540061656265 rpy=-0.252689546175 -0.0085186183214 -0.067039889142
- joint l_upper_arm_mtb_acc_1b12_fixed_joint: origin xyz=-0.0412195 -0.029588 0.0049921 rpy=-1.57079718993 -1.57078381225 2.68257161162 -> xyz=-0.0412194 -0.029588 0.0049921 rpy=-1.57079718993 -1.57078381225 2.68257161162
- joint l_upper_arm_mtb_acc_1b13_fixed_joint: origin xyz=0.010592657 -0.028351 -0.0086914 rpy=-1.57079632657 0.000214520362042 -2.47803674451 -> xyz=0.010592709 -0.028351 -0.0086914 rpy=-1.57079632657 0.000214520362042 -2.47803674451
- joint neck_roll: origin xyz=0.0142999998093 0.0095 0.02080001 rpy=0 0 0 -> xyz=0.0142999998093 0.0095 0.02079997 rpy=0 0 0
- joint neck_yaw: origin xyz=0 -0.022344 -0.02080001 rpy=0 0 0 -> xyz=0 -0.022344 -0.02079997 rpy=0 0 0
- joint r_forearm_mtb_acc_2b7_fixed_joint: origin xyz=-0.0768728106161 0.005497 -0.0110480091994 rpy=0.26179949998 0.000370413042328 1.57125816863 -> xyz=-0.0768727847342 0.005497 -0.0110479126068 rpy=0.26179949998 0.000370413042328 1.57125816863
- joint r_forearm_mtb_acc_2b8_fixed_joint: origin xyz=-0.0514186285381 0.015786 0.0407521034996 rpy=-0.661143946092 0.147825248461 0.092070114703 -> xyz=-0.0514186150796 0.015786 0.0407521537277 rpy=-0.661143946092 0.147825248461 0.092070114703
- joint r_forearm_mtb_acc_2b9_fixed_joint: origin xyz=-0.0216380215578 0.027924 -0.0132491219944 rpy=-1.76682626732 0.261191225646 0.054048344372 -> xyz=-0.0216379956759 0.027924 -0.0132490254018 rpy=-1.76682626732 0.261191225646 0.054048344372
- joint r_forearm_skin_10_fixed_joint: origin xyz=-0.0542285469707 -0.0097861 -0.0321470048792 rpy=-2.94123313406 -0.328304471922 3.1276263754 -> xyz=-0.0542285210888 -0.0097861 -0.0321469082866 rpy=-2.94123313406 -0.328304471922 3.1276263754
- joint r_forearm_skin_11_fixed_joint: origin xyz=-0.0542241170843 0.009043 -0.0321432225378 rpy=2.93929835957 -0.329101389745 -3.12731916446 -> xyz=-0.0542240912024 0.009043 -0.0321431259452 rpy=2.93929835957 -0.329101389745 -3.12731916446
- joint r_forearm_skin_12_fixed_joint: origin xyz=-0.0375994892687 0.018216 -0.0340192145887 rpy=2.58303505964 -0.29483050207 -3.12026580314 -> xyz=-0.0375994633868 0.018216 -0.0340191179961 rpy=2.58303505964 -0.29483050207 -3.12026580314
- joint r_forearm_skin_13_fixed_joint: origin xyz=-0.0228551127224 0.009048 -0.0418919975134 rpy=2.94896679198 -0.270583947189 -3.13981880352 -> xyz=-0.0228550868405 0.009048 -0.0418919009209 rpy=2.94896679198 -0.270583947189 -3.13981880352
- joint r_forearm_skin_14_fixed_joint: origin xyz=-0.0687703535183 0.01716 -0.0230240524437 rpy=2.48044991868 -0.295542566281 -2.91877349139 -> xyz=-0.0687703276364 0.01716 -0.0230239558511 rpy=2.48044991868 -0.295542566281 -2.91877349139
- joint r_forearm_skin_19_fixed_joint: origin xyz=-0.0381266365957 -0.0312941 0.0206905088005 rpy=-1.41560888703 -0.252569290226 3.07715217889 -> xyz=-0.0381266107138 -0.0312941 0.020690605393 rpy=-1.41560888703 -0.252569290226 3.07715217889
- joint r_forearm_skin_1_fixed_joint: origin xyz=-0.0333729194645 0.028826 -0.0198457833637 rpy=1.86694023278 -0.274442533764 -3.09946977984 -> xyz=-0.0333728935826 0.028826 -0.0198456867711 rpy=1.86694023278 -0.274442533764 -3.09946977984
- joint r_forearm_skin_22_fixed_joint: origin xyz=-0.054417420924 -0.0287223 0.0306036550683 rpy=-1.2658242728 -0.234328151379 3.04788317971 -> xyz=-0.0544173950421 -0.0287223 0.0306037516609 rpy=-1.2658242728 -0.234328151379 3.04788317971
- joint r_forearm_skin_24_fixed_joint: origin xyz=-0.0700345474855 -0.0097164 0.0500690507585 rpy=-0.23489327644 -0.0388172993982 3.08676345459 -> xyz=-0.0700345319564 -0.0097164 0.050069108714 rpy=-0.23489327644 -0.0388172993982 3.08676345459
- joint r_forearm_skin_25_fixed_joint: origin xyz=-0.0535999345704 -0.0182238 0.0454697642082 rpy=-0.564295527715 -0.136980272197 3.05963182792 -> xyz=-0.0535999216295 -0.0182238 0.0454698125045 rpy=-0.564295527715 -0.136980272197 3.05963182792
- joint r_forearm_skin_28_fixed_joint: origin xyz=-0.0535859427439 0.017412 0.0453519794414 rpy=0.59077064408 -0.0531607226063 3.10597081167 -> xyz=-0.0535859272148 0.017412 0.045352037397 rpy=0.59077064408 -0.0531607226063 3.10597081167
- joint r_forearm_skin_29_fixed_joint: origin xyz=-0.0700355934441 0.008954 0.050011055327 rpy=0.248630982209 -0.0383136556786 -3.08328999116 -> xyz=-0.0700355805031 0.008954 0.0500111036233 rpy=0.248630982209 -0.0383136556786 -3.08328999116
- joint r_forearm_skin_2_fixed_joint: origin xyz=-0.0146989188671 0.031279 -0.0160118304296 rpy=1.72847287019 -0.264015219116 -3.12733260687 -> xyz=-0.0146988929852 0.031279 -0.0160117338371 rpy=1.72847287019 -0.264015219116 -3.12733260687
- joint r_forearm_skin_3_fixed_joint: origin xyz=-0.0455673195039 -0.030891 -0.00633010588609 rpy=-1.69487280859 -0.269757727104 3.07959743574 -> xyz=-0.045567293622 -0.030891 -0.00633000929351 rpy=-1.69487280859 -0.269757727104 3.07959743574
- joint r_forearm_skin_4_fixed_joint: origin xyz=-0.0635326591815 -0.0281163 -0.00899793917324 rpy=-1.80734960194 -0.0393131796327 2.97997643632 -> xyz=-0.0635326332996 -0.0281163 -0.00899784258066 rpy=-1.80734960194 -0.0393131796327 2.97997643632
- joint r_forearm_skin_6_fixed_joint: origin xyz=-0.0333948695074 -0.0295479 -0.0198326549359 rpy=-1.86628164653 -0.272886336181 3.10448585021 -> xyz=-0.0333948436255 -0.0295479 -0.0198325583433 rpy=-1.86628164653 -0.272886336181 3.10448585021
- joint r_forearm_skin_7_fixed_joint: origin xyz=-0.0147224518893 -0.0319422 -0.0159327448629 rpy=-1.72564640857 -0.263992900722 3.12721254266 -> xyz=-0.0147224260074 -0.0319422 -0.0159326482703 rpy=-1.72564640857 -0.263992900722 3.12721254266
- joint r_hand_dh_frame_fixed_joint: origin xyz=-0.0576543237247 -0.0055568 0.0136937357157 rpy=-1.57079632679 -0.261799319827 3.14159265359 -> xyz=-0.0576542978428 -0.0055568 0.0136938323083 rpy=-1.57079632679 -0.261799319827 3.14159265359
- joint r_shoulder_pitch: origin xyz=-0.120015999809 0.0928 0.0079694 rpy=0 -0.523598883792 3.14159265359 -> xyz=-0.120015999809 0.0928 0.0079693 rpy=0 -0.523598883792 3.14159265359
- joint r_upper_arm_mtb_acc_2b10_fixed_joint: origin xyz=-0.0412195 0.029588 0.0295279 rpy=1.57079546365 1.57078381225 -2.68257161164 -> xyz=-0.0412194 0.029588 0.0295279 rpy=1.57079546365 1.57078381225 -2.68257161164
- joint r_upper_arm_mtb_acc_2b12_fixed_joint: origin xyz=-0.0430555 0.028681 0.0049922 rpy=-1.11177442168 -1.57079632679 0 -> xyz=-0.0430554 0.028681 0.0049922 rpy=-1.11177442168 -1.57079632679 0
- joint r_upper_arm_mtb_acc_2b13_fixed_joint: origin xyz=0.010593184 0.02835 -0.010738 rpy=1.57079632702 -0.000214520362041 2.47803674451 -> xyz=0.010593237 0.02835 -0.010738 rpy=1.57079632702 -0.000214520362041 2.47803674451
- joint torso_roll: origin xyz=0.0270462998093 0.032 -0.0576906 rpy=0 0 0 -> xyz=0.0270462998093 0.032 -0.0573446 rpy=0 0 0
- joint torso_yaw: origin xyz=0 0.05 0.0631871 rpy=0 0 0 -> xyz=0 0.05 0.0628421 rpy=0 0 0
