Commit message: Update dh legacy models to use *_ft for sensor name instead of *_ft_sensor

File: dh/data/legacy_models/headV1-armsV1-legsV1-feetV1/model.urdf (robot description, URDF)
Before this commit: robot iCub, 54 links, 53 joints
Links:
- added link l_arm_ft
- added link l_leg_ft
- added link r_arm_ft
- added link r_leg_ft
Joints:
- added joint l_arm_ft_fixed_joint: type fixed, parent l_upper_arm, child l_arm_ft
- added joint l_leg_ft_fixed_joint: type fixed, parent l_hip_3, child l_leg_ft
- added joint r_arm_ft_fixed_joint: type fixed, parent r_upper_arm, child r_arm_ft
- added joint r_leg_ft_fixed_joint: type fixed, parent r_hip_3, child r_leg_ft

File: dh/data/legacy_models/headV1-armsV1-legsV1-feetV2/model.urdf (robot description, URDF)
Before this commit: robot iCub, 56 links, 55 joints
Links:
- added link l_arm_ft
- added link l_leg_ft
- added link r_arm_ft
- added link r_leg_ft
Joints:
- added joint l_arm_ft_fixed_joint: type fixed, parent l_upper_arm, child l_arm_ft
- added joint l_leg_ft_fixed_joint: type fixed, parent l_hip_3, child l_leg_ft
- added joint r_arm_ft_fixed_joint: type fixed, parent r_upper_arm, child r_arm_ft
- added joint r_leg_ft_fixed_joint: type fixed, parent r_hip_3, child r_leg_ft

File: dh/data/legacy_models/headV1-armsV1-legsV2-feetV1/model.urdf (robot description, URDF)
Before this commit: robot iCub, 54 links, 53 joints
Links:
- added link l_arm_ft
- added link l_leg_ft
- added link r_arm_ft
- added link r_leg_ft
Joints:
- added joint l_arm_ft_fixed_joint: type fixed, parent l_upper_arm, child l_arm_ft
- added joint l_leg_ft_fixed_joint: type fixed, parent l_hip_3, child l_leg_ft
- added joint r_arm_ft_fixed_joint: type fixed, parent r_upper_arm, child r_arm_ft
- added joint r_leg_ft_fixed_joint: type fixed, parent r_hip_3, child r_leg_ft

File: dh/data/legacy_models/headV1-armsV1-legsV2-feetV2/model.urdf (robot description, URDF)
Before this commit: robot iCub, 56 links, 55 joints
Links:
- added link l_arm_ft
- added link l_leg_ft
- added link r_arm_ft
- added link r_leg_ft
Joints:
- added joint l_arm_ft_fixed_joint: type fixed, parent l_upper_arm, child l_arm_ft
- added joint l_leg_ft_fixed_joint: type fixed, parent l_hip_3, child l_leg_ft
- added joint r_arm_ft_fixed_joint: type fixed, parent r_upper_arm, child r_arm_ft
- added joint r_leg_ft_fixed_joint: type fixed, parent r_hip_3, child r_leg_ft

File: dh/data/legacy_models/headV1-armsV2-legsV1-feetV1/model.urdf (robot description, URDF)
Before this commit: robot iCub, 54 links, 53 joints
Links:
- added link l_arm_ft
- added link l_leg_ft
- added link r_arm_ft
- added link r_leg_ft
Joints:
- added joint l_arm_ft_fixed_joint: type fixed, parent l_upper_arm, child l_arm_ft
- added joint l_leg_ft_fixed_joint: type fixed, parent l_hip_3, child l_leg_ft
- added joint r_arm_ft_fixed_joint: type fixed, parent r_upper_arm, child r_arm_ft
- added joint r_leg_ft_fixed_joint: type fixed, parent r_hip_3, child r_leg_ft

File: dh/data/legacy_models/headV2-armsV1-legsV1-feetV1/model.urdf (robot description, URDF)
Before this commit: robot iCub, 54 links, 53 joints
Links:
- added link l_arm_ft
- added link l_leg_ft
- added link r_arm_ft
- added link r_leg_ft
Joints:
- added joint l_arm_ft_fixed_joint: type fixed, parent l_upper_arm, child l_arm_ft
- added joint l_leg_ft_fixed_joint: type fixed, parent l_hip_3, child l_leg_ft
- added joint r_arm_ft_fixed_joint: type fixed, parent r_upper_arm, child r_arm_ft
- added joint r_leg_ft_fixed_joint: type fixed, parent r_hip_3, child r_leg_ft

File: dh/data/legacy_models/headV2-armsV1-legsV1-feetV2/model.urdf (robot description, URDF)
Before this commit: robot iCub, 56 links, 55 joints
Links:
- added link l_arm_ft
- added link l_leg_ft
- added link r_arm_ft
- added link r_leg_ft
Joints:
- added joint l_arm_ft_fixed_joint: type fixed, parent l_upper_arm, child l_arm_ft
- added joint l_leg_ft_fixed_joint: type fixed, parent l_hip_3, child l_leg_ft
- added joint r_arm_ft_fixed_joint: type fixed, parent r_upper_arm, child r_arm_ft
- added joint r_leg_ft_fixed_joint: type fixed, parent r_hip_3, child r_leg_ft

File: dh/data/legacy_models/headV2-armsV1-legsV2-feetV1/model.urdf (robot description, URDF)
Before this commit: robot iCub, 54 links, 53 joints
Links:
- added link l_arm_ft
- added link l_leg_ft
- added link r_arm_ft
- added link r_leg_ft
Joints:
- added joint l_arm_ft_fixed_joint: type fixed, parent l_upper_arm, child l_arm_ft
- added joint l_leg_ft_fixed_joint: type fixed, parent l_hip_3, child l_leg_ft
- added joint r_arm_ft_fixed_joint: type fixed, parent r_upper_arm, child r_arm_ft
- added joint r_leg_ft_fixed_joint: type fixed, parent r_hip_3, child r_leg_ft

File: dh/data/legacy_models/headV2-armsV1-legsV2-feetV2/model.urdf (robot description, URDF)
Before this commit: robot iCub, 56 links, 55 joints
Links:
- added link l_arm_ft
- added link l_leg_ft
- added link r_arm_ft
- added link r_leg_ft
Joints:
- added joint l_arm_ft_fixed_joint: type fixed, parent l_upper_arm, child l_arm_ft
- added joint l_leg_ft_fixed_joint: type fixed, parent l_hip_3, child l_leg_ft
- added joint r_arm_ft_fixed_joint: type fixed, parent r_upper_arm, child r_arm_ft
- added joint r_leg_ft_fixed_joint: type fixed, parent r_hip_3, child r_leg_ft
